File: first/untitled.sch (EAGLE design)
At the start: 13 parts, among them J3 USB_B_PTH

Commit message: fileS
Parts:
- removed C1: 0.8pF, SparkFun-Capacitors:0.8PF-0402-50V-0.1PF
- removed D1, D2: 3.6V, SparkFun-DiscreteSemi:DIODE-ZENER-BZT52C3V6S
- removed J3: USB_B_PTH, SparkFun-Connectors:USB_B_PTH
- removed R1, R2, R3, R4: 0.1, SparkFun-Resistors:0.1OHM-1210-1/2W-1%
- added C2: 0.1uF, SparkFun-Capacitors:0.1UF-KIT-EZ-50V-20%
- added D4, D5: 200mA/100V/1V, SparkFun-DiscreteSemi:DIODE-1N4148
- added J4: (no value), SparkFun-Connectors:USB_AB_SMT
- added R10, R5, R6, R7: 1M, SparkFun-Resistors:1MOHM-HORIZ-1/6W-5%
Connections:
- removed net N$2: D2.C, J3.D+, R4.1
- removed net N$3: D1.C, J3.D-, R1.1, R3.1
- new net N$5: D5.C, J4.D-, R6.1, R7.1
- new net N$6: D4.C, J4.D+, R10.1
- net GND: now also C2.2, D4.A, D5.A, J4.GND; no longer C1.2, D1.A, D2.A, J3.GND, J3.VBUS, R1.2
- net N$1: now also R5.1; no longer R2.1
- net PB3: now also R10.2; no longer R3.2
- net PB4: now also R7.2; no longer R4.2
- net VCC: now also C2.1, J4.VBUS, R5.2, R6.2; no longer C1.1, R2.2

Commit message: fileS
Parts:
- removed R10: 1M, SparkFun-Resistors:1MOHM-HORIZ-1/6W-5%
- added R1: 1k, SparkFun-Resistors:1KOHM-HORIZ-1/4W-1%
Connections:
- net N$5: no longer R6.1
- net N$6: now also R1.1, R6.1; no longer R10.1
- net PB3: now also R1.2; no longer R10.2
Changed lines of the file:
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@@
 <part name="R6" library="SparkFun-Resistors" library_urn="urn:adsk.eagle:library:532" deviceset="1MOHM" device="-HORIZ-1/6W-5%" package3d_urn="urn:adsk.eagle:package:39658/1" value="1M"/>
 <part name="R7" library="SparkFun-Resistors" library_urn="urn:adsk.eagle:library:532" deviceset="1MOHM" device="-HORIZ-1/6W-5%" package3d_urn="urn:adsk.eagle:package:39658/1" value="1M"/>
-<part name="R10" library="SparkFun-Resistors" library_urn="urn:adsk.eagle:library:532" deviceset="1MOHM" device="-HORIZ-1/6W-5%" package3d_urn="urn:adsk.eagle:package:39658/1" value="1M"/>
 <part name="D4" library="SparkFun-DiscreteSemi" library_urn="urn:adsk.eagle:library:514" deviceset="DIODE" device="-1N4148" package3d_urn="urn:adsk.eagle:package:38452/1" value="200mA/100V/1V"/>
 <part name="D5" library="SparkFun-DiscreteSemi" library_urn="urn:adsk.eagle:library:514" deviceset="DIODE" device="-1N4148" package3d_urn="urn:adsk.eagle:package:38452/1" value="200mA/100V/1V"/>
 <part name="J4" library="SparkFun-Connectors" library_urn="urn:adsk.eagle:library:513" deviceset="USB_AB" device="_SMT" package3d_urn="urn:adsk.eagle:package:38266/1"/>
 <part name="C2" library="SparkFun-Capacitors" library_urn="urn:adsk.eagle:library:510" deviceset="0.1UF" device="-KIT-EZ-50V-20%" package3d_urn="urn:adsk.eagle:package:37428/1" value="0.1uF"/>
+<part name="R1" library="SparkFun-Resistors" library_urn="urn:adsk.eagle:library:532" deviceset="1KOHM" device="-HORIZ-1/4W-1%" package3d_urn="urn:adsk.eagle:package:39658/1" value="1k"/>
 </parts>
 <sheets>
@@
 <instance part="R6" gate="G$1" x="106.68" y="-10.16" rot="R90"/>
 <instance part="R7" gate="G$1" x="144.78" y="-22.86"/>
-<instance part="R10" gate="G$1" x="129.54" y="-20.32"/>
 <instance part="D4" gate="G$1" x="99.06" y="-38.1" rot="R90"/>
 <instance part="D5" gate="G$1" x="111.76" y="-38.1" rot="R90"/>
 <instance part="J4" gate="G$1" x="55.88" y="-22.86" rot="R180"/>
 <instance part="C2" gate="G$1" x="48.26" y="48.26"/>
+<instance part="R1" gate="G$1" x="129.54" y="-20.32"/>
 </instances>
 <busses>
@@
 <segment>
 <wire x1="134.62" y1="-20.32" x2="160.02" y2="-20.32" width="0.1524" layer="91"/>
-<pinref part="R10" gate="G$1" pin="2"/>
+<pinref part="R1" gate="G$1" pin="2"/>
 </segment>
 </net>
@@
 </segment>
 </net>
-<net name="N$2" class="0">
-<segment>
-<wire x1="111.76" y1="-20.32" x2="106.68" y2="-20.32" width="0.1524" layer="91"/>
-</segment>
-</net>
 <net name="N$5" class="0">
 <segment>
-<wire x1="66.04" y1="-22.86" x2="106.68" y2="-22.86" width="0.1524" layer="91"/>
-<wire x1="106.68" y1="-22.86" x2="111.76" y2="-22.86" width="0.1524" layer="91"/>
+<wire x1="66.04" y1="-22.86" x2="111.76" y2="-22.86" width="0.1524" layer="91"/>
 <wire x1="111.76" y1="-22.86" x2="139.7" y2="-22.86" width="0.1524" layer="91"/>
 <wire x1="111.76" y1="-35.56" x2="111.76" y2="-22.86" width="0.1524" layer="91"/>
 <junction x="111.76" y="-22.86"/>
-<wire x1="106.68" y1="-15.24" x2="106.68" y2="-22.86" width="0.1524" layer="91"/>
-<junction x="106.68" y="-22.86"/>
-<pinref part="R6" gate="G$1" pin="1"/>
 <pinref part="R7" gate="G$1" pin="1"/>
 <pinref part="D5" gate="G$1" pin="C"/>
@@
 <segment>
 <wire x1="68.58" y1="-20.32" x2="99.06" y2="-20.32" width="0.1524" layer="91"/>
-<wire x1="99.06" y1="-20.32" x2="124.46" y2="-20.32" width="0.1524" layer="91"/>
 <wire x1="99.06" y1="-35.56" x2="99.06" y2="-20.32" width="0.1524" layer="91"/>
-<junction x="99.06" y="-20.32"/>
-<pinref part="R10" gate="G$1" pin="1"/>
 <pinref part="D4" gate="G$1" pin="C"/>
 <wire x1="68.58" y1="-20.32" x2="68.58" y2="-25.4" width="0.1524" layer="91"/>
@@
 <pinref part="J4" gate="G$1" pin="D+"/>
 <wire x1="63.5" y1="-22.86" x2="60.96" y2="-22.86" width="0.1524" layer="91"/>
-</segment>
-</net>
+<pinref part="R1" gate="G$1" pin="1"/>
+<wire x1="124.46" y1="-20.32" x2="106.68" y2="-20.32" width="0.1524" layer="91"/>
+<junction x="99.06" y="-20.32"/>
+<pinref part="R6" gate="G$1" pin="1"/>
+<wire x1="106.68" y1="-20.32" x2="99.06" y2="-20.32" width="0.1524" layer="91"/>
+<wire x1="106.68" y1="-15.24" x2="106.68" y2="-20.32" width="0.1524" layer="91"/>
+<junction x="106.68" y="-20.32"/>
+</segment>
+</net>

Commit message: fileS
Changed lines of the file:
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@@
+</segment>
+<segment>
+<pinref part="J2" gate="G$1" pin="4"/>
+<wire x1="35.56" y1="-12.7" x2="45.72" y2="-12.7" width="0.1524" layer="91"/>
+<label x="38.1" y="-12.7" size="1.778" layer="95"/>
 </segment>
 <segment>
@@
 <wire x1="2.54" y1="73.66" x2="-5.08" y2="73.66" width="0.1524" layer="91"/>
 <junction x="2.54" y="73.66"/>
-<label x="-5.08" y="73.66" size="1.778" layer="95"/>
-</segment>
-<segment>
-<pinref part="J2" gate="G$1" pin="4"/>
-<wire x1="35.56" y1="-12.7" x2="45.72" y2="-12.7" width="0.1524" layer="91"/>
-<label x="38.1" y="-12.7" size="1.778" layer="95"/>
+<label x="-10.16" y="73.66" size="1.778" layer="95"/>
 </segment>
 </net>
