File: first/untitled.brd (EAGLE design)
At the start: 160 x 100 mm, 13 parts, among them J3 USB_B_PTH

Commit message: fileS
Parts:
- removed C1: 0.8pF, SparkFun-Capacitors:0402
- removed D1, D2: 3.6V, SparkFun-DiscreteSemi:SOD-323
- removed J3: USB_B_PTH, SparkFun-Connectors:USB-B-PTH
- removed R1, R2, R3, R4: 0.1, SparkFun-Resistors:1210
- added C2: 0.1uF, SparkFun-Capacitors:CAP-PTH-SMALL-KIT
- added D4, D5: 200mA/100V/1V, SparkFun-DiscreteSemi:DIODE-1N4148
- added J4: (no value), SparkFun-Connectors:USB-AB-MICRO-SMD
- added R10, R5, R6, R7: 1M, SparkFun-Resistors:AXIAL-0.3
- moved U$2 174.1 mm to (132.1, 67.3), turned to 90 degrees
- moved J2 162.7 mm to (127.0, 54.6)
- moved J1 154.3 mm to (127.0, 69.8)
- moved S1 146.7 mm to (119.4, 62.2)
- moved D3 130.5 mm to (90.2, 62.2)
Connections:
- removed net N$2: D2.C, J3.D+, R4.1
- removed net N$3: D1.C, J3.D-, R1.1, R3.1
- new net N$5: D5.C, J4.D-1, R6.P$1, R7.P$1
- new net N$6: D4.C, J4.D+1, R10.P$1
- net GND: now also C2.2, D4.A, D5.A, J4.GND1; no longer C1.2, D1.A, D2.A, J3.GND, J3.VBUS, R1.2
- net N$1: now also R5.P$1; no longer R2.1
- net PB3: now also R10.P$2; no longer R3.2
- net PB4: now also R7.P$2; no longer R4.2
- net VCC: now also C2.1, J4.VBUS1, R5.P$2, R6.P$2; no longer C1.1, R2.2
Routing:
- net N$4: track 0.00 -> 200.7 mm

Commit message: fileS
Parts:
- moved R6 12.7 mm to (105.4, 73.7)
- moved R7 11.7 mm to (114.3, 68.6)
- moved S1 5.08 mm to (124.5, 62.2)
- moved R5 4.02 mm to (108.0, 55.9)
- moved J1 3.81 mm to (130.8, 69.8)
- moved J2 3.81 mm to (130.8, 54.6)
- moved U$2 3.81 mm to (135.9, 67.3)
Changed lines of the file:
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@@
 <elements>
 <element name="D3" library="SparkFun-LED" library_urn="urn:adsk.eagle:library:529" package="LED_3MM-NS" package3d_urn="urn:adsk.eagle:package:39356/1" value="" x="90.17" y="62.23"/>
-<element name="J1" library="SparkFun-Connectors" library_urn="urn:adsk.eagle:library:513" package="1X04" package3d_urn="urn:adsk.eagle:package:38085/1" value="" x="127" y="69.85">
-<attribute name="PROD_ID" value="CONN-09696" x="127" y="69.85" size="1.778" layer="27" display="off"/>
+<element name="J1" library="SparkFun-Connectors" library_urn="urn:adsk.eagle:library:513" package="1X04" package3d_urn="urn:adsk.eagle:package:38085/1" value="" x="130.81" y="69.85">
+<attribute name="PROD_ID" value="CONN-09696" x="130.81" y="69.85" size="1.778" layer="27" display="off"/>
 </element>
-<element name="J2" library="SparkFun-Connectors" library_urn="urn:adsk.eagle:library:513" package="1X04" package3d_urn="urn:adsk.eagle:package:38085/1" value="" x="127" y="54.61">
-<attribute name="PROD_ID" value="CONN-09696" x="127" y="54.61" size="1.778" layer="27" display="off"/>
+<element name="J2" library="SparkFun-Connectors" library_urn="urn:adsk.eagle:library:513" package="1X04" package3d_urn="urn:adsk.eagle:package:38085/1" value="" x="130.81" y="54.61">
+<attribute name="PROD_ID" value="CONN-09696" x="130.81" y="54.61" size="1.778" layer="27" display="off"/>
 </element>
-<element name="S1" library="SparkFun-Switches" library_urn="urn:adsk.eagle:library:535" package="TACTILE_SWITCH_PTH_6.0MM" package3d_urn="urn:adsk.eagle:package:40163/1" value="MOMENTARY-SWITCH-SPST-PTH-6.0MM" x="119.38" y="62.23">
-<attribute name="PROD_ID" value=" SWCH-08441" x="119.38" y="62.23" size="1.778" layer="27" display="off"/>
-<attribute name="SF_SKU" value="COM-00097" x="119.38" y="62.23" size="1.778" layer="27" display="off"/>
+<element name="S1" library="SparkFun-Switches" library_urn="urn:adsk.eagle:library:535" package="TACTILE_SWITCH_PTH_6.0MM" package3d_urn="urn:adsk.eagle:package:40163/1" value="MOMENTARY-SWITCH-SPST-PTH-6.0MM" x="124.46" y="62.23">
+<attribute name="PROD_ID" value=" SWCH-08441" x="124.46" y="62.23" size="1.778" layer="27" display="off"/>
+<attribute name="SF_SKU" value="COM-00097" x="124.46" y="62.23" size="1.778" layer="27" display="off"/>
 </element>
-<element name="U$2" library="whatamIdoing" package="DIP8" value="ATINY85" x="132.08" y="67.31" rot="R90"/>
-<element name="R5" library="SparkFun-Resistors" library_urn="urn:adsk.eagle:library:532" package="AXIAL-0.3" package3d_urn="urn:adsk.eagle:package:39658/1" value="1M" x="104.14" y="54.61">
-<attribute name="PROD_ID" value="RES-09559" x="104.14" y="54.61" size="1.778" layer="27" display="off"/>
+<element name="U$2" library="whatamIdoing" package="DIP8" value="ATINY85" x="135.89" y="67.31" rot="R90"/>
+<element name="R5" library="SparkFun-Resistors" library_urn="urn:adsk.eagle:library:532" package="AXIAL-0.3" package3d_urn="urn:adsk.eagle:package:39658/1" value="1M" x="107.95" y="55.88">
+<attribute name="PROD_ID" value="RES-09559" x="107.95" y="55.88" size="1.778" layer="27" display="off"/>
 </element>
-<element name="R6" library="SparkFun-Resistors" library_urn="urn:adsk.eagle:library:532" package="AXIAL-0.3" package3d_urn="urn:adsk.eagle:package:39658/1" value="1M" x="105.41" y="60.96">
-<attribute name="PROD_ID" value="RES-09559" x="105.41" y="60.96" size="1.778" layer="27" display="off"/>
+<element name="R6" library="SparkFun-Resistors" library_urn="urn:adsk.eagle:library:532" package="AXIAL-0.3" package3d_urn="urn:adsk.eagle:package:39658/1" value="1M" x="105.41" y="73.66">
+<attribute name="PROD_ID" value="RES-09559" x="105.41" y="73.66" size="1.778" layer="27" display="off"/>
 </element>
-<element name="R7" library="SparkFun-Resistors" library_urn="urn:adsk.eagle:library:532" package="AXIAL-0.3" package3d_urn="urn:adsk.eagle:package:39658/1" value="1M" x="102.87" y="71.12">
-<attribute name="PROD_ID" value="RES-09559" x="102.87" y="71.12" size="1.778" layer="27" display="off"/>
+<element name="R7" library="SparkFun-Resistors" library_urn="urn:adsk.eagle:library:532" package="AXIAL-0.3" package3d_urn="urn:adsk.eagle:package:39658/1" value="1M" x="114.3" y="68.58">
+<attribute name="PROD_ID" value="RES-09559" x="114.3" y="68.58" size="1.778" layer="27" display="off"/>
 </element>
 <element name="R10" library="SparkFun-Resistors" library_urn="urn:adsk.eagle:library:532" package="AXIAL-0.3" package3d_urn="urn:adsk.eagle:package:39658/1" value="1M" x="105.41" y="49.53">
@@
 <contactref element="J4" pad="VBUS1"/>
 <contactref element="C2" pad="1"/>
-<wire x1="127" y1="67.31" x2="127" y2="69.85" width="0" layer="19" extent="1-1"/>
-<wire x1="109.22" y1="60.96" x2="127" y2="67.31" width="0" layer="19" extent="1-1"/>
-<wire x1="107.95" y1="54.61" x2="109.22" y2="60.96" width="0" layer="19" extent="1-1"/>
-<wire x1="78.9" y1="62.26" x2="107.95" y2="54.61" width="0" layer="19" extent="1-1"/>
+<wire x1="130.81" y1="67.31" x2="130.81" y2="69.85" width="0" layer="19" extent="1-1"/>
+<wire x1="109.22" y1="73.66" x2="130.81" y2="67.31" width="0" layer="19" extent="1-1"/>
+<wire x1="111.76" y1="55.88" x2="109.22" y2="73.66" width="0" layer="19" extent="1-1"/>
+<wire x1="78.9" y1="62.26" x2="111.76" y2="55.88" width="0" layer="19" extent="1-1"/>
 <wire x1="83.693" y1="50.8" x2="78.9" y2="62.26" width="0" layer="19" extent="1-1"/>
 </signal>
@@
 <contactref element="J4" pad="GND1"/>
 <contactref element="C2" pad="2"/>
-<wire x1="127" y1="54.61" x2="134.62" y2="57.15" width="0" layer="19" extent="1-1"/>
-<wire x1="116.1288" y1="59.9694" x2="127" y2="54.61" width="0" layer="19" extent="1-1"/>
-<wire x1="80.01" y1="73.66" x2="116.1288" y2="59.9694" width="0" layer="19" extent="1-1"/>
+<wire x1="130.81" y1="54.61" x2="138.43" y2="57.15" width="0" layer="19" extent="1-1"/>
+<wire x1="121.2088" y1="59.9694" x2="130.81" y2="54.61" width="0" layer="19" extent="1-1"/>
+<wire x1="80.01" y1="73.66" x2="121.2088" y2="59.9694" width="0" layer="19" extent="1-1"/>
 <wire x1="86.36" y1="55.88" x2="80.01" y2="73.66" width="0" layer="19" extent="1-1"/>
 <wire x1="78.9" y1="59.66" x2="86.36" y2="55.88" width="0" layer="19" extent="1-1"/>
@@
 <contactref element="U$2" pad="P$5"/>
 <contactref element="J1" pad="4"/>
-<wire x1="134.62" y1="69.85" x2="134.62" y2="67.31" width="0" layer="19" extent="1-1"/>
+<wire x1="138.43" y1="69.85" x2="138.43" y2="67.31" width="0" layer="19" extent="1-1"/>
 </signal>
 <signal name="PB1">
 <contactref element="U$2" pad="P$6"/>
 <contactref element="J1" pad="3"/>
-<wire x1="132.08" y1="69.85" x2="132.08" y2="67.31" width="0" layer="19" extent="1-1"/>
+<wire x1="135.89" y1="69.85" x2="135.89" y2="67.31" width="0" layer="19" extent="1-1"/>
 </signal>
 <signal name="PB2">
 <contactref element="U$2" pad="P$7"/>
 <contactref element="J1" pad="2"/>
-<wire x1="129.54" y1="69.85" x2="129.54" y2="67.31" width="0" layer="19" extent="1-1"/>
+<wire x1="133.35" y1="69.85" x2="133.35" y2="67.31" width="0" layer="19" extent="1-1"/>
 </signal>
 <signal name="PB3">
@@
 <contactref element="J2" pad="3"/>
 <contactref element="R10" pad="P$2"/>
-<wire x1="132.08" y1="54.61" x2="129.54" y2="57.15" width="0" layer="19" extent="1-1"/>
-<wire x1="109.22" y1="49.53" x2="129.54" y2="57.15" width="0" layer="19" extent="1-1"/>
+<wire x1="135.89" y1="54.61" x2="133.35" y2="57.15" width="0" layer="19" extent="1-1"/>
+<wire x1="109.22" y1="49.53" x2="133.35" y2="57.15" width="0" layer="19" extent="1-1"/>
 </signal>
 <signal name="PB4">
@@
 <contactref element="J2" pad="2"/>
 <contactref element="R7" pad="P$2"/>
-<wire x1="129.54" y1="54.61" x2="132.08" y2="57.15" width="0" layer="19" extent="1-1"/>
-<wire x1="106.68" y1="71.12" x2="129.54" y2="54.61" width="0" layer="19" extent="1-1"/>
+<wire x1="133.35" y1="54.61" x2="135.89" y2="57.15" width="0" layer="19" extent="1-1"/>
+<wire x1="118.11" y1="68.58" x2="133.35" y2="54.61" width="0" layer="19" extent="1-1"/>
 </signal>
 <signal name="RESET">
@@
 <contactref element="D3" pad="K"/>
 <contactref element="J2" pad="4"/>
-<wire x1="91.44" y1="62.23" x2="127" y2="57.15" width="0" layer="19" extent="1-1"/>
-<wire x1="116.1288" y1="64.4906" x2="91.44" y2="62.23" width="0" layer="19" extent="1-1"/>
-<wire x1="134.62" y1="54.61" x2="116.1288" y2="64.4906" width="0" layer="19" extent="1-1"/>
+<wire x1="91.44" y1="62.23" x2="130.81" y2="57.15" width="0" layer="19" extent="1-1"/>
+<wire x1="121.2088" y1="64.4906" x2="91.44" y2="62.23" width="0" layer="19" extent="1-1"/>
+<wire x1="138.43" y1="54.61" x2="121.2088" y2="64.4906" width="0" layer="19" extent="1-1"/>
 </signal>
 <signal name="N$1">
 <contactref element="D3" pad="A"/>
 <contactref element="R5" pad="P$1"/>
-<wire x1="100.33" y1="54.61" x2="88.9" y2="62.23" width="0" layer="19" extent="1-1"/>
+<wire x1="104.14" y1="55.88" x2="88.9" y2="62.23" width="0" layer="19" extent="1-1"/>
 </signal>
 <signal name="N$4">
@@
 <contactref element="D5" pad="C"/>
 <contactref element="J4" pad="D-1"/>
-<wire x1="101.6" y1="60.96" x2="99.06" y2="71.12" width="0" layer="19" extent="1-1"/>
-<wire x1="93.98" y1="55.88" x2="101.6" y2="60.96" width="0" layer="19" extent="1-1"/>
+<wire x1="101.6" y1="73.66" x2="110.49" y2="68.58" width="0" layer="19" extent="1-1"/>
+<wire x1="93.98" y1="55.88" x2="101.6" y2="73.66" width="0" layer="19" extent="1-1"/>
 <wire x1="78.9" y1="61.61" x2="93.98" y2="55.88" width="0" layer="19" extent="1-1"/>
 </signal>

Commit message: fileS
Parts:
- removed R10: 1M, SparkFun-Resistors:AXIAL-0.3
- added R1: 1k, SparkFun-Resistors:AXIAL-0.3
- moved C2 58.3 mm to (142.2, 62.2), turned to 90 degrees
- moved D5 23.7 mm to (113.0, 62.2), turned to 90 degrees
- moved D3 22.9 mm to (111.8, 69.8), turned to 180 degrees
- moved D4 21.1 mm to (101.6, 62.2), turned to 90 degrees
- moved R5 19.8 mm to (121.9, 69.8)
- moved R6 12.0 mm to (109.2, 62.2), turned to 270 degrees
- moved J4 11.5 mm to (87.6, 62.2)
- moved R7 6.84 mm to (116.8, 62.2), turned to 90 degrees
- turned S1 to 180 degrees
Connections:
- net N$5: no longer R6.P$1
- net N$6: now also R1.P$1, R6.P$1; no longer R10.P$1
- net PB3: now also R1.P$2; no longer R10.P$2
Routing:
- net N$4: track 200.7 -> 160.0 mm
- net N$6: track 0.00 -> 7.62 mm
- net VCC: track 0.00 -> 5.08 mm
- net N$1: track 0.00 -> 5.08 mm

Commit message: fileS
Parts:
- moved J2 7.62 mm to (138.4, 54.6), turned to 180 degrees
- turned R7 to 270 degrees
Routing:
- net PB2: track 0.00 -> 2.54 mm
- net PB1: track 0.00 -> 2.54 mm
- net PB0: track 0.00 -> 2.54 mm
Changed lines of the file:
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@@
 <attribute name="PROD_ID" value="CONN-09696" x="130.81" y="69.85" size="1.778" layer="27" display="off"/>
 </element>
-<element name="J2" library="SparkFun-Connectors" library_urn="urn:adsk.eagle:library:513" package="1X04" package3d_urn="urn:adsk.eagle:package:38085/1" value="" x="130.81" y="54.61">
-<attribute name="PROD_ID" value="CONN-09696" x="130.81" y="54.61" size="1.778" layer="27" display="off"/>
+<element name="J2" library="SparkFun-Connectors" library_urn="urn:adsk.eagle:library:513" package="1X04" package3d_urn="urn:adsk.eagle:package:38085/1" value="" x="138.43" y="54.61" rot="R180">
+<attribute name="PROD_ID" value="CONN-09696" x="138.43" y="54.61" size="1.778" layer="27" rot="R180" display="off"/>
 </element>
 <element name="S1" library="SparkFun-Switches" library_urn="urn:adsk.eagle:library:535" package="TACTILE_SWITCH_PTH_6.0MM" package3d_urn="urn:adsk.eagle:package:40163/1" value="MOMENTARY-SWITCH-SPST-PTH-6.0MM" x="124.46" y="62.23" rot="R180">
@@
 <attribute name="PROD_ID" value="RES-09559" x="109.22" y="62.23" size="1.778" layer="27" rot="R270" display="off"/>
 </element>
-<element name="R7" library="SparkFun-Resistors" library_urn="urn:adsk.eagle:library:532" package="AXIAL-0.3" package3d_urn="urn:adsk.eagle:package:39658/1" value="1M" x="116.84" y="62.23" rot="R90">
-<attribute name="PROD_ID" value="RES-09559" x="116.84" y="62.23" size="1.778" layer="27" rot="R90" display="off"/>
+<element name="R7" library="SparkFun-Resistors" library_urn="urn:adsk.eagle:library:532" package="AXIAL-0.3" package3d_urn="urn:adsk.eagle:package:39658/1" value="1M" x="116.84" y="62.23" rot="R270">
+<attribute name="PROD_ID" value="RES-09559" x="116.84" y="62.23" size="1.778" layer="27" rot="R270" display="off"/>
 </element>
 <element name="D4" library="SparkFun-DiscreteSemi" library_urn="urn:adsk.eagle:library:514" package="DIODE-1N4148" package3d_urn="urn:adsk.eagle:package:38452/1" value="200mA/100V/1V" x="101.6" y="62.23" rot="R90">
@@
 <contactref element="J4" pad="GND1"/>
 <contactref element="C2" pad="2"/>
-<wire x1="130.81" y1="54.61" x2="138.43" y2="57.15" width="0" layer="19" extent="1-1"/>
-<wire x1="127.7112" y1="64.4906" x2="130.81" y2="54.61" width="0" layer="19" extent="1-1"/>
-<wire x1="101.6" y1="58.42" x2="127.7112" y2="64.4906" width="0" layer="19" extent="1-1"/>
-<wire x1="113.03" y1="58.42" x2="101.6" y2="58.42" width="0" layer="19" extent="1-1"/>
-<wire x1="90.33" y1="60.93" x2="113.03" y2="58.42" width="0" layer="19" extent="1-1"/>
-<wire x1="142.24" y1="63.627" x2="90.33" y2="60.93" width="0" layer="19" extent="1-1"/>
+<wire x1="135.15265625" y1="55.7784" x2="134.1326" y2="56.79845625" width="0" layer="19" extent="1-16"/>
+<wire x1="134.1326" y1="56.79845625" x2="134.1326" y2="58.0692" width="0" layer="19" extent="1-16"/>
+<wire x1="138.91396875" y1="55.7784" x2="135.15265625" y2="55.7784" width="0" layer="19" extent="1-16"/>
+<wire x1="134.1326" y1="58.0692" x2="127.7112" y2="64.4906" width="0" layer="19" extent="1-16"/>
+<wire x1="139.5984" y1="54.12603125" x2="139.5984" y2="55.09396875" width="0" layer="19" extent="1-16"/>
+<wire x1="139.5984" y1="55.09396875" x2="138.91396875" y2="55.7784" width="0" layer="19" extent="1-16"/>
+<wire x1="133.17083125" y1="53.1368" x2="138.60916875" y2="53.1368" width="0" layer="19" extent="1-16"/>
+<wire x1="138.60916875" y1="53.1368" x2="139.5984" y2="54.12603125" width="0" layer="19" extent="1-16"/>
+<wire x1="138.43" y1="54.61" x2="131.69763125" y2="54.61" width="0" layer="19" extent="1-16"/>
+<wire x1="131.69763125" y1="54.61" x2="133.17083125" y2="53.1368" width="0" layer="19" extent="1-16"/>
+<wire x1="138.91396875" y1="55.7784" x2="138.43" y2="56.26236875" width="0" layer="19" extent="1-16"/>
+<wire x1="138.43" y1="56.26236875" x2="138.43" y2="57.15" width="0" layer="19" extent="1-16"/>
+<wire x1="138.43" y1="57.15" x2="138.43" y2="60.96" width="0" layer="19" extent="1-16"/>
+<wire x1="138.43" y1="60.96" x2="139.7" y2="62.23" width="0" layer="19" extent="1-16"/>
+<wire x1="139.7" y1="62.23" x2="139.7" y2="63.5" width="0" layer="19" extent="1-16"/>
+<wire x1="139.7" y1="63.5" x2="139.827" y2="63.627" width="0" layer="19" extent="1-16"/>
+<wire x1="139.827" y1="63.627" x2="142.24" y2="63.627" width="0" layer="19" extent="1-16"/>
+<wire x1="113.03" y1="58.42" x2="127.7112" y2="64.4906" width="0" layer="19" extent="1-1"/>
+<wire x1="101.6" y1="58.42" x2="113.03" y2="58.42" width="0" layer="19" extent="1-1"/>
+<wire x1="90.33" y1="60.93" x2="101.6" y2="58.42" width="0" layer="19" extent="1-1"/>
 </signal>
 <signal name="PB0">
 <contactref element="U$2" pad="P$5"/>
 <contactref element="J1" pad="4"/>
-<wire x1="138.43" y1="69.85" x2="138.43" y2="67.31" width="0" layer="19" extent="1-1"/>
+<wire x1="138.43" y1="69.85" x2="138.43" y2="67.31" width="0.1524" layer="1"/>
 </signal>
 <signal name="PB1">
 <contactref element="U$2" pad="P$6"/>
 <contactref element="J1" pad="3"/>
-<wire x1="135.89" y1="69.85" x2="135.89" y2="67.31" width="0" layer="19" extent="1-1"/>
+<wire x1="135.89" y1="69.85" x2="135.89" y2="67.31" width="0.1524" layer="1"/>
 </signal>
 <signal name="PB2">
 <contactref element="U$2" pad="P$7"/>
 <contactref element="J1" pad="2"/>
-<wire x1="133.35" y1="69.85" x2="133.35" y2="67.31" width="0" layer="19" extent="1-1"/>
+<wire x1="133.35" y1="69.85" x2="133.35" y2="67.31" width="0.1524" layer="1"/>
 </signal>
 <signal name="PB3">
@@
 <contactref element="J2" pad="3"/>
 <contactref element="R1" pad="P$2"/>
-<wire x1="135.89" y1="54.61" x2="133.35" y2="57.15" width="0" layer="19" extent="1-1"/>
-<wire x1="105.41" y1="58.42" x2="133.35" y2="57.15" width="0" layer="19" extent="1-1"/>
+<wire x1="107.56763125" y1="58.42" x2="105.41" y2="58.42" width="0" layer="19" extent="1-16"/>
+<wire x1="108.73603125" y1="57.2516" x2="107.56763125" y2="58.42" width="0" layer="19" extent="1-16"/>
+<wire x1="113.51396875" y1="57.2516" x2="108.73603125" y2="57.2516" width="0" layer="19" extent="1-16"/>
+<wire x1="129.3622" y1="61.1378" x2="127.22723125" y2="61.1378" width="0" layer="19" extent="1-16"/>
+<wire x1="117.32396875" y1="59.5884" x2="115.85076875" y2="59.5884" width="0" layer="19" extent="1-16"/>
+<wire x1="115.85076875" y1="59.5884" x2="113.51396875" y2="57.2516" width="0" layer="19" extent="1-16"/>
+<wire x1="118.11136875" y1="58.801" x2="117.32396875" y2="59.5884" width="0" layer="19" extent="1-16"/>
+<wire x1="124.89043125" y1="58.801" x2="118.11136875" y2="58.801" width="0" layer="19" extent="1-16"/>
+<wire x1="127.22723125" y1="61.1378" x2="124.89043125" y2="58.801" width="0" layer="19" extent="1-16"/>
+<wire x1="133.35" y1="54.61" x2="129.3622" y2="61.1378" width="0" layer="19" extent="1-16"/>
+<wire x1="133.35" y1="54.61" x2="133.35" y2="57.15" width="0" layer="19" extent="1-1"/>
 </signal>
 <signal name="PB4">
@@
 <contactref element="J2" pad="2"/>
 <contactref element="R7" pad="P$2"/>
-<wire x1="133.35" y1="54.61" x2="135.89" y2="57.15" width="0" layer="19" extent="1-1"/>
-<wire x1="116.84" y1="66.04" x2="133.35" y2="54.61" width="0" layer="19" extent="1-1"/>
+<wire x1="135.89" y1="54.61" x2="132.4864" y2="55.4736" width="0" layer="19" extent="1-16"/>
+<wire x1="132.4864" y1="55.4736" x2="131.77594375" y2="55.4736" width="0" layer="19" extent="1-16"/>
+<wire x1="130.88214375" y1="56.3674" x2="130.1613125" y2="56.3674" width="0" layer="19" extent="1-16"/>
+<wire x1="131.77594375" y1="55.4736" x2="130.88214375" y2="56.3674" width="0" layer="19" extent="1-16"/>
+<wire x1="128.1087125" y1="58.42" x2="116.84" y2="58.42" width="0" layer="19" extent="1-16"/>
+<wire x1="130.1613125" y1="56.3674" x2="128.1087125" y2="58.42" width="0" layer="19" extent="1-16"/>
+<wire x1="135.89" y1="54.61" x2="135.89" y2="57.15" width="0" layer="19" extent="1-1"/>
 </signal>
 <signal name="RESET">
 <contactref element="U$2" pad="P$1"/>
+<contactref element="J2" pad="4"/>
 <contactref element="S1" pad="1"/>
 <contactref element="D3" pad="K"/>
-<contactref element="J2" pad="4"/>
-<wire x1="110.49" y1="69.85" x2="130.81" y2="57.15" width="0" layer="19" extent="1-1"/>
-<wire x1="127.7112" y1="59.9694" x2="110.49" y2="69.85" width="0" layer="19" extent="1-1"/>
-<wire x1="138.43" y1="54.61" x2="127.7112" y2="59.9694" width="0" layer="19" extent="1-1"/>
+<wire x1="136.37396875" y1="53.4416" x2="135.40603125" y2="53.4416" width="0" layer="19" extent="1-16"/>
+<wire x1="134.5184" y1="55.09396875" x2="133.83396875" y2="55.7784" width="0" layer="19" extent="1-16"/>
+<wire x1="130.81" y1="54.61" x2="137.54236875" y2="54.61" width="0" layer="19" extent="1-16"/>
+<wire x1="131.9022" y1="55.7784" x2="127.7112" y2="59.9694" width="0" layer="19" extent="1-16"/>
+<wire x1="137.54236875" y1="54.61" x2="136.37396875" y2="53.4416" width="0" layer="19" extent="1-16"/>
+<wire x1="133.83396875" y1="55.7784" x2="131.9022" y2="55.7784" width="0" layer="19" extent="1-16"/>
+<wire x1="135.40603125" y1="53.4416" x2="134.5184" y2="54.32923125" width="0" layer="19" extent="1-16"/>
+<wire x1="134.5184" y1="54.32923125" x2="134.5184" y2="55.09396875" width="0" layer="19" extent="1-16"/>
+<wire x1="131.9022" y1="55.7784" x2="130.81" y2="57.15" width="0" layer="19" extent="1-1"/>
+<wire x1="110.49" y1="69.85" x2="127.7112" y2="59.9694" width="0" layer="19" extent="1-1"/>
 </signal>
 <signal name="N$1">
@@
 <contactref element="D5" pad="C"/>
 <contactref element="J4" pad="D-1"/>
-<wire x1="116.84" y1="58.42" x2="113.03" y2="66.04" width="0" layer="19" extent="1-1"/>
+<wire x1="116.84" y1="66.04" x2="113.03" y2="66.04" width="0" layer="19" extent="1-1"/>
 <wire x1="90.33" y1="62.88" x2="113.03" y2="66.04" width="0" layer="19" extent="1-1"/>
 </signal>
