File: first/untitled.brd (EAGLE design)
At the start: 160 x 100 mm, 13 parts

Commit message: fileS
Routing:
- net GND: track 0.00 -> 47.5 mm
- net PB3: track 0.00 -> 39.4 mm
- net PB4: track 0.00 -> 26.2 mm
- net RESET: track 0.00 -> 8.29 mm
- net VCC: track 5.08 -> 7.62 mm
Changed lines of the file:
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@@
 <contactref element="C2" pad="1"/>
 <wire x1="130.81" y1="69.85" x2="125.73" y2="69.85" width="0.1524" layer="1"/>
+<wire x1="130.81" y1="69.85" x2="130.81" y2="67.31" width="0.1524" layer="1"/>
 <wire x1="130.81" y1="67.31" x2="142.24" y2="60.833" width="0" layer="19" extent="1-1"/>
-<wire x1="130.81" y1="69.85" x2="130.81" y2="67.31" width="0" layer="19" extent="1-1"/>
 <wire x1="109.22" y1="58.42" x2="125.73" y2="69.85" width="0" layer="19" extent="1-1"/>
 <wire x1="90.33" y1="63.53" x2="109.22" y2="58.42" width="0" layer="19" extent="1-1"/>
@@
 <contactref element="J4" pad="GND1"/>
 <contactref element="C2" pad="2"/>
-<wire x1="135.15265625" y1="55.7784" x2="134.1326" y2="56.79845625" width="0" layer="19" extent="1-16"/>
-<wire x1="134.1326" y1="56.79845625" x2="134.1326" y2="58.0692" width="0" layer="19" extent="1-16"/>
-<wire x1="138.91396875" y1="55.7784" x2="135.15265625" y2="55.7784" width="0" layer="19" extent="1-16"/>
-<wire x1="134.1326" y1="58.0692" x2="127.7112" y2="64.4906" width="0" layer="19" extent="1-16"/>
-<wire x1="139.5984" y1="54.12603125" x2="139.5984" y2="55.09396875" width="0" layer="19" extent="1-16"/>
-<wire x1="139.5984" y1="55.09396875" x2="138.91396875" y2="55.7784" width="0" layer="19" extent="1-16"/>
-<wire x1="133.17083125" y1="53.1368" x2="138.60916875" y2="53.1368" width="0" layer="19" extent="1-16"/>
-<wire x1="138.60916875" y1="53.1368" x2="139.5984" y2="54.12603125" width="0" layer="19" extent="1-16"/>
-<wire x1="138.43" y1="54.61" x2="131.69763125" y2="54.61" width="0" layer="19" extent="1-16"/>
-<wire x1="131.69763125" y1="54.61" x2="133.17083125" y2="53.1368" width="0" layer="19" extent="1-16"/>
-<wire x1="138.91396875" y1="55.7784" x2="138.43" y2="56.26236875" width="0" layer="19" extent="1-16"/>
-<wire x1="138.43" y1="56.26236875" x2="138.43" y2="57.15" width="0" layer="19" extent="1-16"/>
-<wire x1="138.43" y1="57.15" x2="138.43" y2="60.96" width="0" layer="19" extent="1-16"/>
-<wire x1="138.43" y1="60.96" x2="139.7" y2="62.23" width="0" layer="19" extent="1-16"/>
-<wire x1="139.7" y1="62.23" x2="139.7" y2="63.5" width="0" layer="19" extent="1-16"/>
-<wire x1="139.7" y1="63.5" x2="139.827" y2="63.627" width="0" layer="19" extent="1-16"/>
-<wire x1="139.827" y1="63.627" x2="142.24" y2="63.627" width="0" layer="19" extent="1-16"/>
+<wire x1="138.43" y1="54.61" x2="138.43" y2="57.15" width="0.1524" layer="1"/>
+<wire x1="138.43" y1="57.15" x2="138.43" y2="63.5" width="0.1524" layer="1"/>
+<wire x1="138.43" y1="63.5" x2="138.557" y2="63.627" width="0.1524" layer="1"/>
+<wire x1="138.557" y1="63.627" x2="142.24" y2="63.627" width="0.1524" layer="1"/>
+<wire x1="138.43" y1="63.5" x2="137.4394" y2="64.4906" width="0.1524" layer="1"/>
+<wire x1="137.4394" y1="64.4906" x2="127.7112" y2="64.4906" width="0.1524" layer="1"/>
+<wire x1="113.03" y1="58.42" x2="110.87236875" y2="58.42" width="0.1524" layer="1"/>
+<wire x1="103.75763125" y1="58.42" x2="101.6" y2="58.42" width="0.1524" layer="1"/>
+<wire x1="110.87236875" y1="58.42" x2="109.70396875" y2="57.2516" width="0.1524" layer="1"/>
+<wire x1="104.92603125" y1="57.2516" x2="103.75763125" y2="58.42" width="0.1524" layer="1"/>
+<wire x1="109.70396875" y1="57.2516" x2="104.92603125" y2="57.2516" width="0.1524" layer="1"/>
+<wire x1="101.6" y1="58.42" x2="99.06" y2="60.96" width="0.1524" layer="1"/>
+<wire x1="99.06" y1="60.96" x2="91.44" y2="60.96" width="0.1524" layer="1"/>
 <wire x1="113.03" y1="58.42" x2="127.7112" y2="64.4906" width="0" layer="19" extent="1-1"/>
-<wire x1="101.6" y1="58.42" x2="113.03" y2="58.42" width="0" layer="19" extent="1-1"/>
-<wire x1="90.33" y1="60.93" x2="101.6" y2="58.42" width="0" layer="19" extent="1-1"/>
+<wire x1="90.33" y1="60.93" x2="91.44" y2="60.96" width="0" layer="19" extent="1-1"/>
 </signal>
 <signal name="PB0">
@@
 <contactref element="J2" pad="3"/>
 <contactref element="R1" pad="P$2"/>
-<wire x1="107.56763125" y1="58.42" x2="105.41" y2="58.42" width="0" layer="19" extent="1-16"/>
-<wire x1="108.73603125" y1="57.2516" x2="107.56763125" y2="58.42" width="0" layer="19" extent="1-16"/>
-<wire x1="113.51396875" y1="57.2516" x2="108.73603125" y2="57.2516" width="0" layer="19" extent="1-16"/>
-<wire x1="129.3622" y1="61.1378" x2="127.22723125" y2="61.1378" width="0" layer="19" extent="1-16"/>
-<wire x1="117.32396875" y1="59.5884" x2="115.85076875" y2="59.5884" width="0" layer="19" extent="1-16"/>
-<wire x1="115.85076875" y1="59.5884" x2="113.51396875" y2="57.2516" width="0" layer="19" extent="1-16"/>
-<wire x1="118.11136875" y1="58.801" x2="117.32396875" y2="59.5884" width="0" layer="19" extent="1-16"/>
-<wire x1="124.89043125" y1="58.801" x2="118.11136875" y2="58.801" width="0" layer="19" extent="1-16"/>
-<wire x1="127.22723125" y1="61.1378" x2="124.89043125" y2="58.801" width="0" layer="19" extent="1-16"/>
-<wire x1="133.35" y1="54.61" x2="129.3622" y2="61.1378" width="0" layer="19" extent="1-16"/>
-<wire x1="133.35" y1="54.61" x2="133.35" y2="57.15" width="0" layer="19" extent="1-1"/>
+<wire x1="133.35" y1="54.61" x2="133.35" y2="57.15" width="0.1524" layer="1"/>
+<wire x1="133.35" y1="57.15" x2="133.35" y2="62.23" width="0.1524" layer="1"/>
+<wire x1="133.35" y1="62.23" x2="105.41" y2="62.23" width="0.1524" layer="1"/>
+<wire x1="105.41" y1="62.23" x2="105.41" y2="58.42" width="0.1524" layer="1"/>
 </signal>
 <signal name="PB4">
@@
 <contactref element="J2" pad="2"/>
 <contactref element="R7" pad="P$2"/>
-<wire x1="135.89" y1="54.61" x2="132.4864" y2="55.4736" width="0" layer="19" extent="1-16"/>
-<wire x1="132.4864" y1="55.4736" x2="131.77594375" y2="55.4736" width="0" layer="19" extent="1-16"/>
-<wire x1="130.88214375" y1="56.3674" x2="130.1613125" y2="56.3674" width="0" layer="19" extent="1-16"/>
-<wire x1="131.77594375" y1="55.4736" x2="130.88214375" y2="56.3674" width="0" layer="19" extent="1-16"/>
-<wire x1="128.1087125" y1="58.42" x2="116.84" y2="58.42" width="0" layer="19" extent="1-16"/>
-<wire x1="130.1613125" y1="56.3674" x2="128.1087125" y2="58.42" width="0" layer="19" extent="1-16"/>
-<wire x1="135.89" y1="54.61" x2="135.89" y2="57.15" width="0" layer="19" extent="1-1"/>
+<wire x1="135.89" y1="54.61" x2="135.89" y2="57.15" width="0.1524" layer="1"/>
+<wire x1="134.5184" y1="54.12603125" x2="133.83396875" y2="53.4416" width="0.1524" layer="1"/>
+<wire x1="133.83396875" y1="53.4416" x2="121.8184" y2="53.4416" width="0.1524" layer="1"/>
+<wire x1="135.89" y1="57.15" x2="134.5184" y2="55.7784" width="0.1524" layer="1"/>
+<wire x1="134.5184" y1="55.7784" x2="134.5184" y2="54.12603125" width="0.1524" layer="1"/>
+<wire x1="121.8184" y1="53.4416" x2="116.84" y2="58.42" width="0.1524" layer="1"/>
 </signal>
 <signal name="RESET">
@@
 <contactref element="S1" pad="1"/>
 <contactref element="D3" pad="K"/>
-<wire x1="136.37396875" y1="53.4416" x2="135.40603125" y2="53.4416" width="0" layer="19" extent="1-16"/>
-<wire x1="134.5184" y1="55.09396875" x2="133.83396875" y2="55.7784" width="0" layer="19" extent="1-16"/>
-<wire x1="130.81" y1="54.61" x2="137.54236875" y2="54.61" width="0" layer="19" extent="1-16"/>
-<wire x1="131.9022" y1="55.7784" x2="127.7112" y2="59.9694" width="0" layer="19" extent="1-16"/>
-<wire x1="137.54236875" y1="54.61" x2="136.37396875" y2="53.4416" width="0" layer="19" extent="1-16"/>
-<wire x1="133.83396875" y1="55.7784" x2="131.9022" y2="55.7784" width="0" layer="19" extent="1-16"/>
-<wire x1="135.40603125" y1="53.4416" x2="134.5184" y2="54.32923125" width="0" layer="19" extent="1-16"/>
-<wire x1="134.5184" y1="54.32923125" x2="134.5184" y2="55.09396875" width="0" layer="19" extent="1-16"/>
-<wire x1="131.9022" y1="55.7784" x2="130.81" y2="57.15" width="0" layer="19" extent="1-1"/>
+<wire x1="130.81" y1="54.61" x2="130.81" y2="57.15" width="0.1524" layer="1"/>
+<wire x1="130.81" y1="57.15" x2="130.81" y2="59.69" width="0.1524" layer="1"/>
+<wire x1="130.81" y1="59.69" x2="130.5306" y2="59.9694" width="0.1524" layer="1"/>
+<wire x1="130.5306" y1="59.9694" x2="127.7112" y2="59.9694" width="0.1524" layer="1"/>
 <wire x1="110.49" y1="69.85" x2="127.7112" y2="59.9694" width="0" layer="19" extent="1-1"/>
 </signal>

Commit message: badges
Routing:
- net GND: track 47.5 -> 0.00 mm
- net PB3: track 39.4 -> 0.00 mm
- net PB4: track 26.2 -> 0.00 mm
- net RESET: track 8.29 -> 0.00 mm
- net N$6: track 7.62 -> 0.00 mm
- net VCC: track 7.62 -> 0.18 mm
- net N$1: track 5.08 -> 0.00 mm
- net PB2: track 2.54 -> 0.00 mm
- net PB1: track 2.54 -> 0.00 mm
- net PB0: track 2.54 -> 0.00 mm
- net N$5: track 0.00 -> 0.77 mm

Commit message: LED attack
Routing:
- net GND: track 0.00 -> 57.2 mm
- net N$5: track 0.77 -> 3.81 mm
Changed lines of the file:
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@@
 <contactref element="J4" pad="GND1"/>
 <contactref element="C2" pad="2"/>
-<wire x1="138.43" y1="54.61" x2="138.43" y2="57.15" width="0" layer="19" extent="1-16"/>
-<wire x1="138.43" y1="57.15" x2="138.43" y2="63.5" width="0" layer="19" extent="1-16"/>
-<wire x1="138.43" y1="63.5" x2="138.557" y2="63.627" width="0" layer="19" extent="1-16"/>
-<wire x1="138.557" y1="63.627" x2="142.24" y2="63.627" width="0" layer="19" extent="1-16"/>
-<wire x1="138.43" y1="63.5" x2="137.4394" y2="64.4906" width="0" layer="19" extent="1-16"/>
-<wire x1="137.4394" y1="64.4906" x2="127.7112" y2="64.4906" width="0" layer="19" extent="1-16"/>
-<wire x1="113.03" y1="58.42" x2="110.87236875" y2="58.42" width="0" layer="19" extent="1-16"/>
-<wire x1="103.75763125" y1="58.42" x2="101.6" y2="58.42" width="0" layer="19" extent="1-16"/>
-<wire x1="110.87236875" y1="58.42" x2="109.70396875" y2="57.2516" width="0" layer="19" extent="1-16"/>
-<wire x1="104.92603125" y1="57.2516" x2="103.75763125" y2="58.42" width="0" layer="19" extent="1-16"/>
-<wire x1="109.70396875" y1="57.2516" x2="104.92603125" y2="57.2516" width="0" layer="19" extent="1-16"/>
-<wire x1="101.6" y1="58.42" x2="99.06" y2="60.96" width="0" layer="19" extent="1-16"/>
-<wire x1="99.06" y1="60.96" x2="91.44" y2="60.96" width="0" layer="19" extent="1-16"/>
-<wire x1="127.7112" y1="64.4906" x2="129.667" y2="62.5348" width="0" layer="19" extent="1-16"/>
-<wire x1="129.667" y1="62.5348" x2="133.47625625" y2="62.5348" width="0" layer="19" extent="1-16"/>
-<wire x1="133.47625625" y1="62.5348" x2="137.16" y2="58.85105625" width="0" layer="19" extent="1-16"/>
-<wire x1="137.16" y1="58.85105625" x2="137.16" y2="53.34" width="0" layer="19" extent="1-16"/>
-<wire x1="137.16" y1="53.34" x2="134.163425" y2="53.34" width="0" layer="19" extent="1-16"/>
-<wire x1="134.163425" y1="53.34" x2="133.960225" y2="53.1368" width="0" layer="19" extent="1-16"/>
-<wire x1="133.960225" y1="53.1368" x2="121.69214375" y2="53.1368" width="0" layer="19" extent="1-16"/>
-<wire x1="117.67894375" y1="57.15" x2="113.03" y2="57.15" width="0" layer="19" extent="1-16"/>
-<wire x1="113.03" y1="57.15" x2="113.03" y2="58.42" width="0" layer="19" extent="1-16"/>
-<wire x1="121.69214375" y1="53.1368" x2="117.67894375" y2="57.15" width="0" layer="19" extent="1-16"/>
-<wire x1="90.33" y1="60.93" x2="91.44" y2="60.96" width="0" layer="19" extent="1-1"/>
+<wire x1="127.7112" y1="64.4906" x2="129.9718" y2="62.23" width="0.1524" layer="1"/>
+<wire x1="129.9718" y1="62.23" x2="133.35" y2="62.23" width="0.1524" layer="1"/>
+<wire x1="133.35" y1="62.23" x2="137.16" y2="58.42" width="0.1524" layer="1"/>
+<wire x1="137.16" y1="58.42" x2="137.16" y2="53.34" width="0.1524" layer="1"/>
+<wire x1="137.16" y1="53.34" x2="121.92" y2="53.34" width="0.1524" layer="1"/>
+<wire x1="121.92" y1="53.34" x2="118.11" y2="57.15" width="0.1524" layer="1"/>
+<wire x1="118.11" y1="57.15" x2="113.03" y2="57.15" width="0.1524" layer="1"/>
+<wire x1="113.03" y1="57.15" x2="113.03" y2="58.42" width="0.1524" layer="1"/>
+<wire x1="113.03" y1="58.42" x2="111.76" y2="57.15" width="0.1524" layer="1"/>
+<wire x1="111.76" y1="57.15" x2="101.6" y2="57.15" width="0.1524" layer="1"/>
+<wire x1="101.6" y1="57.15" x2="101.6" y2="58.42" width="0.1524" layer="1"/>
+<wire x1="137.16" y1="58.42" x2="142.24" y2="63.627" width="0" layer="19" extent="1-1"/>
+<wire x1="138.43" y1="57.15" x2="137.16" y2="58.42" width="0" layer="19" extent="1-1"/>
+<wire x1="138.43" y1="54.61" x2="137.16" y2="53.34" width="0" layer="19" extent="1-1"/>
+<wire x1="101.6" y1="58.42" x2="90.33" y2="60.93" width="0" layer="19" extent="1-1"/>
 </signal>
 <signal name="PB0">
@@
 <contactref element="D5" pad="C"/>
 <contactref element="J4" pad="D-1"/>
-<wire x1="116.84" y1="66.04" x2="113.03" y2="66.04" width="0" layer="19" extent="1-16"/>
-<wire x1="91.1246875" y1="63.1014" x2="90.94705" y2="63.1014" width="0.1524" layer="1"/>
-<wire x1="90.94705" y1="63.1014" x2="90.527825" y2="62.682175" width="0.1524" layer="1"/>
-<wire x1="113.03" y1="66.04" x2="110.87236875" y2="66.04" width="0" layer="19" extent="1-16"/>
-<wire x1="110.87236875" y1="66.04" x2="109.70396875" y2="67.2084" width="0" layer="19" extent="1-16"/>
-<wire x1="109.70396875" y1="67.2084" x2="95.2316875" y2="67.2084" width="0" layer="19" extent="1-16"/>
-<wire x1="95.2316875" y1="67.2084" x2="91.1246875" y2="63.1014" width="0" layer="19" extent="1-16"/>
-<wire x1="90.527825" y1="62.682175" x2="90.33" y2="62.88" width="0" layer="19" extent="1-1"/>
+<wire x1="91.1246875" y1="63.1014" x2="90.94705" y2="63.1014" width="0" layer="19" extent="1-16"/>
+<wire x1="90.527825" y1="62.682175" x2="90.94705" y2="63.1014" width="0" layer="19" extent="1-16"/>
+<wire x1="116.84" y1="66.04" x2="113.03" y2="66.04" width="0.1524" layer="1"/>
+<wire x1="90.33" y1="62.88" x2="91.1246875" y2="63.1014" width="0" layer="19" extent="1-16"/>
+<wire x1="113.03" y1="66.04" x2="91.1246875" y2="63.1014" width="0" layer="19" extent="1-1"/>
 </signal>
 <signal name="N$6">
