File: charbadge/charLED.sch (EAGLE design)
At the start: 7 parts, among them U1 ATTINY85-20P

Commit message: char badge
Parts:
- removed D2, D3, D4, D5: (no value), SparkFun-LED:LED3MM
- added LED1, LED2, LED3, LED4: (no value), adafruit:LED5MM
- added R1, R2, R3, R4: 100k, SparkFun-Resistors:100KOHM-HORIZ-1/4W-1%
Connections:
- new net N$2: LED1.A, R2.1
- new net N$7: LED2.A, R4.1
- new net N$8: LED4.A, R3.1
- new net N$9: LED3.A, R1.1
- net N$1: now also LED1.C, LED2.C; no longer D2.C, D3.C
- net N$4: now also LED3.C, LED4.C; no longer D4.C, D5.C
- net N$6: now also R1.2, R2.2, R3.2, R4.2; no longer D2.A, D3.A, D4.A, D5.A
Changed lines of the file:
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@@
 <parts>
 <part name="U1" library="_hhn_attiny25_45_85" deviceset="ATTINY85*" device="P" technology="-20"/>
-<part name="D2" library="SparkFun-LED" library_urn="urn:adsk.eagle:library:529" deviceset="LED" device="3MM" package3d_urn="urn:adsk.eagle:package:39361/1"/>
-<part name="D3" library="SparkFun-LED" library_urn="urn:adsk.eagle:library:529" deviceset="LED" device="3MM" package3d_urn="urn:adsk.eagle:package:39361/1"/>
-<part name="D4" library="SparkFun-LED" library_urn="urn:adsk.eagle:library:529" deviceset="LED" device="3MM" package3d_urn="urn:adsk.eagle:package:39361/1"/>
-<part name="D5" library="SparkFun-LED" library_urn="urn:adsk.eagle:library:529" deviceset="LED" device="3MM" package3d_urn="urn:adsk.eagle:package:39361/1"/>
 <part name="S1" library="adafruit" deviceset="EG1218" device="S"/>
 <part name="BT1" library="SparkFun-Batteries" library_urn="urn:adsk.eagle:library:508" deviceset="BATTERY" device="-20MM_PTH" package3d_urn="urn:adsk.eagle:package:37214/1"/>
+<part name="LED1" library="adafruit" deviceset="LED" device="5MM"/>
+<part name="LED2" library="adafruit" deviceset="LED" device="5MM"/>
+<part name="LED3" library="adafruit" deviceset="LED" device="5MM"/>
+<part name="LED4" library="adafruit" deviceset="LED" device="5MM"/>
+<part name="R1" library="SparkFun-Resistors" library_urn="urn:adsk.eagle:library:532" deviceset="100KOHM" device="-HORIZ-1/4W-1%" package3d_urn="urn:adsk.eagle:package:39658/1" value="100k"/>
+<part name="R2" library="SparkFun-Resistors" library_urn="urn:adsk.eagle:library:532" deviceset="100KOHM" device="-HORIZ-1/4W-1%" package3d_urn="urn:adsk.eagle:package:39658/1" value="100k"/>
+<part name="R3" library="SparkFun-Resistors" library_urn="urn:adsk.eagle:library:532" deviceset="100KOHM" device="-HORIZ-1/4W-1%" package3d_urn="urn:adsk.eagle:package:39658/1" value="100k"/>
+<part name="R4" library="SparkFun-Resistors" library_urn="urn:adsk.eagle:library:532" deviceset="100KOHM" device="-HORIZ-1/4W-1%" package3d_urn="urn:adsk.eagle:package:39658/1" value="100k"/>
 </parts>
 <sheets>
@@
 <instances>
 <instance part="U1" gate="G$1" x="63.5" y="60.96"/>
-<instance part="D2" gate="G$1" x="106.68" y="71.12"/>
-<instance part="D3" gate="G$1" x="116.84" y="71.12"/>
-<instance part="D4" gate="G$1" x="127" y="71.12"/>
-<instance part="D5" gate="G$1" x="137.16" y="71.12"/>
 <instance part="S1" gate="1" x="30.48" y="27.94" rot="R180"/>
 <instance part="BT1" gate="G$1" x="35.56" y="-12.7" rot="R180"/>
+<instance part="LED1" gate="G$1" x="106.68" y="71.12"/>
+<instance part="LED2" gate="G$1" x="116.84" y="71.12"/>
+<instance part="LED3" gate="G$1" x="127" y="71.12"/>
+<instance part="LED4" gate="G$1" x="137.16" y="71.12"/>
+<instance part="R1" gate="G$1" x="127" y="81.28" rot="R90"/>
+<instance part="R2" gate="G$1" x="106.68" y="81.28" rot="R90"/>
+<instance part="R3" gate="G$1" x="137.16" y="81.28" rot="R90"/>
+<instance part="R4" gate="G$1" x="116.84" y="81.28" rot="R90"/>
 </instances>
 <busses>
@@
 <pinref part="U1" gate="G$1" pin="PB0"/>
 <wire x1="81.28" y1="53.34" x2="127" y2="53.34" width="0.1524" layer="91"/>
-<pinref part="D4" gate="G$1" pin="C"/>
 <wire x1="127" y1="53.34" x2="127" y2="66.04" width="0.1524" layer="91"/>
 <wire x1="127" y1="53.34" x2="137.16" y2="53.34" width="0.1524" layer="91"/>
 <junction x="127" y="53.34"/>
-<pinref part="D5" gate="G$1" pin="C"/>
 <wire x1="137.16" y1="53.34" x2="137.16" y2="66.04" width="0.1524" layer="91"/>
+<pinref part="LED3" gate="G$1" pin="C"/>
+<pinref part="LED4" gate="G$1" pin="C"/>
 </segment>
 </net>
@@
 <junction x="27.94" y="66.04"/>
 <wire x1="27.94" y1="88.9" x2="106.68" y2="88.9" width="0.1524" layer="91"/>
-<pinref part="D5" gate="G$1" pin="A"/>
 <wire x1="106.68" y1="88.9" x2="116.84" y2="88.9" width="0.1524" layer="91"/>
 <wire x1="116.84" y1="88.9" x2="127" y2="88.9" width="0.1524" layer="91"/>
 <wire x1="127" y1="88.9" x2="137.16" y2="88.9" width="0.1524" layer="91"/>
-<wire x1="137.16" y1="88.9" x2="137.16" y2="73.66" width="0.1524" layer="91"/>
-<pinref part="D4" gate="G$1" pin="A"/>
-<wire x1="127" y1="73.66" x2="127" y2="88.9" width="0.1524" layer="91"/>
+<pinref part="R2" gate="G$1" pin="2"/>
+<wire x1="106.68" y1="86.36" x2="106.68" y2="88.9" width="0.1524" layer="91"/>
+<junction x="106.68" y="88.9"/>
+<pinref part="R4" gate="G$1" pin="2"/>
+<wire x1="116.84" y1="86.36" x2="116.84" y2="88.9" width="0.1524" layer="91"/>
+<junction x="116.84" y="88.9"/>
+<pinref part="R1" gate="G$1" pin="2"/>
+<wire x1="127" y1="86.36" x2="127" y2="88.9" width="0.1524" layer="91"/>
 <junction x="127" y="88.9"/>
-<pinref part="D3" gate="G$1" pin="A"/>
-<wire x1="116.84" y1="73.66" x2="116.84" y2="88.9" width="0.1524" layer="91"/>
-<pinref part="D2" gate="G$1" pin="A"/>
-<wire x1="106.68" y1="73.66" x2="106.68" y2="88.9" width="0.1524" layer="91"/>
+<pinref part="R3" gate="G$1" pin="2"/>
+<wire x1="137.16" y1="86.36" x2="137.16" y2="88.9" width="0.1524" layer="91"/>
 </segment>
 </net>
@@
 <segment>
 <pinref part="U1" gate="G$1" pin="PB1"/>
-<pinref part="D2" gate="G$1" pin="C"/>
 <wire x1="81.28" y1="55.88" x2="106.68" y2="55.88" width="0.1524" layer="91"/>
 <wire x1="106.68" y1="55.88" x2="106.68" y2="66.04" width="0.1524" layer="91"/>
-<pinref part="D3" gate="G$1" pin="C"/>
 <wire x1="106.68" y1="55.88" x2="116.84" y2="55.88" width="0.1524" layer="91"/>
 <wire x1="116.84" y1="55.88" x2="116.84" y2="66.04" width="0.1524" layer="91"/>
 <junction x="106.68" y="55.88"/>
+<pinref part="LED1" gate="G$1" pin="C"/>
+<pinref part="LED2" gate="G$1" pin="C"/>
 </segment>
 </net>
+<net name="N$2" class="0">
+<segment>
+<pinref part="R2" gate="G$1" pin="1"/>
+<pinref part="LED1" gate="G$1" pin="A"/>
+<wire x1="106.68" y1="76.2" x2="106.68" y2="73.66" width="0.1524" layer="91"/>
+</segment>
+</net>
+<net name="N$7" class="0">
+<segment>
+<pinref part="LED2" gate="G$1" pin="A"/>
+<pinref part="R4" gate="G$1" pin="1"/>
+<wire x1="116.84" y1="73.66" x2="116.84" y2="76.2" width="0.1524" layer="91"/>
+</segment>
+</net>
+<net name="N$8" class="0">
+<segment>
+<pinref part="R3" gate="G$1" pin="1"/>
+<pinref part="LED4" gate="G$1" pin="A"/>
+<wire x1="137.16" y1="76.2" x2="137.16" y2="73.66" width="0.1524" layer="91"/>
+</segment>
+</net>
+<net name="N$9" class="0">
+<segment>
+<pinref part="R1" gate="G$1" pin="1"/>
+<pinref part="LED3" gate="G$1" pin="A"/>
+<wire x1="127" y1="76.2" x2="127" y2="73.66" width="0.1524" layer="91"/>
+</segment>
+</net>
