File: charbadge/charLED.brd (EAGLE design)
At the start: 143.2 x 143.2 mm, 7 parts, among them U1 ATTINY85-20P

Commit message: char badge
Parts:
- removed D2, D3, D4, D5: (no value), SparkFun-LED:LED_3MM
- added LED1, LED2, LED3, LED4: (no value), adafruit:LED5MM
- added R1, R2, R3, R4: 100k, SparkFun-Resistors:AXIAL-0.3
- moved BT1 91.2 mm to (111.1, 32.9), flipped to the bottom, turned to 89.9 degrees
- moved S1 83.6 mm to (38.0, 3.22), turned to 179.7 degrees
- moved U1 45.6 mm to (22.6, 16.6), turned to 90 degrees
Connections:
- new net N$2: LED1.A, R2.P$1
- new net N$7: LED2.A, R4.P$1
- new net N$8: LED4.A, R3.P$1
- new net N$9: LED3.A, R1.P$1
- net N$1: now also LED1.K, LED2.K; no longer D2.K, D3.K
- net N$4: now also LED3.K, LED4.K; no longer D4.K, D5.K
- net N$6: now also R1.P$2, R2.P$2, R3.P$2, R4.P$2; no longer D2.A, D3.A, D4.A, D5.A
Routing:
- net N$6: track 0.00 -> 191.4 mm
- net N$10: track 0.00 -> 154.2 mm, vias 0 -> 1
- net N$5: track 0.00 -> 100.1 mm
- net N$3: track 0.00 -> 79.5 mm
- net N$4: track 0.00 -> 65.2 mm
- net N$1: track 0.00 -> 63.8 mm
- net N$8: track 0.00 -> 11.5 mm
- net N$2: track 0.00 -> 6.24 mm
- net N$7: track 0.00 -> 5.16 mm
- net N$9: track 0.00 -> 4.25 mm
Other:
- board text added: "https://github.com/littlefoot22/badges/tree/master/charbadge"

Commit message: char badge
Routing:
- net N$10: track 154.2 -> 0.00 mm, vias 1 -> 0
- net N$6: track 191.4 -> 190.5 mm
Other:
- board text removed: "/Users/chrisbuckner/badges/charbadge/char5in_mask_new_no tail_bmp.bmp"
- board text removed: "/Users/chrisbuckner/badges/charbadge/char5in_mask_new_no tail_bmp_silk.bmp"
Changed lines of the file:
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@@
 <rectangle x1="29.591" y1="102.06558125" x2="38.735" y2="102.15041875" layer="29"/>
 <rectangle x1="29.591" y1="102.15041875" x2="38.735" y2="102.235" layer="29"/>
-<text x="0" y="-0.42418125" size="0.17018125" layer="29" font="vector">/Users/chrisbuckner/badges/charbadge/char5in_mask_new_no tail_bmp.bmp</text>
 <rectangle x1="47.54118125" y1="15.45158125" x2="49.657" y2="15.53641875" layer="21"/>
 <rectangle x1="47.54118125" y1="15.53641875" x2="49.657" y2="15.621" layer="21"/>
@@
 <rectangle x1="21.463" y1="111.29441875" x2="22.90318125" y2="111.379" layer="21"/>
 <rectangle x1="21.463" y1="111.379" x2="22.90318125" y2="111.46358125" layer="21"/>
-<text x="0" y="-0.42418125" size="0.17018125" layer="21" font="vector">/Users/chrisbuckner/badges/charbadge/char5in_mask_new_no tail_bmp_silk.bmp</text>
 <rectangle x1="39.07281875" y1="26.797" x2="41.61281875" y2="26.88158125" layer="1"/>
 <rectangle x1="51.435" y1="26.797" x2="56.43118125" y2="26.88158125" layer="1"/>
@@
 <rectangle x1="29.591" y1="102.06558125" x2="38.735" y2="102.15041875" layer="1"/>
 <rectangle x1="29.591" y1="102.15041875" x2="38.735" y2="102.235" layer="1"/>
-<text x="0" y="-0.42418125" size="0.17018125" layer="1" font="vector">/Users/chrisbuckner/badges/charbadge/char5in_mask_new_no tail_bmp.bmp</text>
 <circle x="64.170915625" y="60.5306125" radius="71.61568125" width="0.1524" layer="20"/>
-<text x="98.118853125" y="-0.761921875" size="1.27" layer="22" font="vector" rot="MR0">https://github.com/littlefoot22/badges/tree/master/charbadge</text>
+<text x="37.080296875" y="8.719790625" size="1.27" layer="21" font="vector">https://github.com/littlefoot22/badges/tree/master/charbadge</text>
 </plain>
 <attributes>
@@
 <wire x1="31.619646875" y1="3.343809375" x2="28.360496875" y2="3.343809375" width="0.1524" layer="1"/>
 <wire x1="28.360496875" y1="3.343809375" x2="28.23331875" y2="3.343809375" width="0.1524" layer="1"/>
-<wire x1="24.97416875" y1="3.343809375" x2="23.323140625" y2="3.343809375" width="0.1524" layer="1"/>
-<wire x1="23.873609375" y1="3.894278125" x2="23.323140625" y2="3.343809375" width="0.1524" layer="1"/>
-<wire x1="23.873609375" y1="3.894278125" x2="6.687996875" y2="21.079890625" width="0.1524" layer="1"/>
-<wire x1="6.687996875" y1="21.079890625" x2="6.687996875" y2="42.498415625" width="0.1524" layer="1"/>
+<wire x1="24.0007875" y1="3.343809375" x2="6.687996875" y2="20.6566" width="0.1524" layer="1"/>
+<wire x1="6.687996875" y1="20.6566" x2="6.687996875" y2="42.498415625" width="0.1524" layer="1"/>
 <wire x1="6.687996875" y1="42.498415625" x2="6.687996875" y2="42.66773125" width="0.1524" layer="1"/>
 <wire x1="6.687996875" y1="42.66773125" x2="6.687996875" y2="51.641121875" width="0.1524" layer="1"/>
@@
 <wire x1="2.878378125" y1="62.477753125" x2="6.18005" y2="65.779425" width="0.1524" layer="1"/>
 <wire x1="22.434425" y1="50.118034375" x2="22.51908125" y2="50.033378125" width="0.1524" layer="1"/>
+<wire x1="24.97416875" y1="3.343809375" x2="24.0007875" y2="3.343809375" width="0.1524" layer="1"/>
 </signal>
 <signal name="N$1">
@@
 <wire x1="16.846978125" y1="53.58825625" x2="19.132753125" y2="55.87403125" width="0.1524" layer="1"/>
 </signal>
-<signal name="N$10">
+<signal name="N$11">
 <via x="66.033396875" y="128.426490625" extent="1-16" drill="1"/>
-<wire x1="66.033396875" y1="128.426490625" x2="65.440790625" y2="127.833884375" width="0.1524" layer="1"/>
-<wire x1="66.0334" y1="128.42649375" x2="65.440790625" y2="127.833884375" width="0.1524" layer="1"/>
-<wire x1="59.17608125" y1="121.569175" x2="33.270671875" y2="121.569175" width="0.1524" layer="1"/>
-<wire x1="33.270671875" y1="121.569175" x2="33.016696875" y2="121.3152" width="0.1524" layer="1"/>
-<wire x1="66.033396875" y1="128.426490625" x2="73.1446875" y2="121.3152" width="0.1524" layer="1"/>
-<wire x1="73.1446875" y1="121.3152" x2="96.425690625" y2="121.3152" width="0.1524" layer="1"/>
-<wire x1="96.425690625" y1="121.3152" x2="96.679665625" y2="121.061225" width="0.1524" layer="1"/>
-<wire x1="96.679665625" y1="121.061225" x2="96.679665625" y2="112.680065625" width="0.1524" layer="1"/>
-<wire x1="96.679665625" y1="112.680065625" x2="96.679665625" y2="112.59540625" width="0.1524" layer="1"/>
-<wire x1="66.0334" y1="128.42649375" x2="66.0334" y2="101.92846875" width="0.1524" layer="1"/>
-<wire x1="66.0334" y1="101.92846875" x2="73.314" y2="94.64786875" width="0.1524" layer="1"/>
-<wire x1="65.440790625" y1="127.833884375" x2="59.17608125" y2="121.569175" width="0.1524" layer="1"/>
-<wire x1="33.016696875" y1="109.801684375" x2="32.932040625" y2="109.717028125" width="0.1524" layer="1"/>
-<wire x1="33.016696875" y1="121.3152" x2="33.016696875" y2="109.801684375" width="0.1524" layer="1"/>
-<wire x1="73.314" y1="94.64786875" x2="73.314" y2="86.77465625" width="0.1524" layer="1"/>
-<wire x1="73.314" y1="86.77465625" x2="80.34063125" y2="79.748025" width="0.1524" layer="1"/>
-<wire x1="96.679665625" y1="112.680065625" x2="96.679665625" y2="103.70629375" width="0.1524" layer="1"/>
 </signal>
 </signals>

Commit message: char badge
Parts:
- moved S1 24.5 mm to (62.5, 3.30)
Routing:
- net N$3: track 79.5 -> 61.4 mm
- net N$6: track 190.5 -> 205.0 mm
- net N$5: track 100.1 -> 105.6 mm
Changed lines of the file:
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@@
 <attribute name="SF_SKU" value="PRT-00783" x="111.068896875" y="32.93318125" size="1.778" layer="28" rot="MR89.9" display="off"/>
 </element>
-<element name="S1" library="adafruit" package="EG1218" value="" x="38.00785" y="3.219553125" rot="R179.7"/>
+<element name="S1" library="adafruit" package="EG1218" value="" x="62.47406875" y="3.304209375" rot="R179.7"/>
 <element name="U1" library="_hhn_attiny25_45_85" package="PDIP08_300MIL" value="ATTINY85-20P" x="22.601325" y="16.595803125" rot="R90"/>
 <element name="LED1" library="adafruit" package="LED5MM" value="" x="14.8151875" y="68.996425" rot="R269.9"/>
@@
 <contactref element="S1" pad="O"/>
 <contactref element="BT1" pad="2"/>
-<wire x1="89.49528125" y1="3.19535" x2="40.63766875" y2="3.19535" width="0.1524" layer="1"/>
-<wire x1="111.083121875" y1="24.783190625" x2="89.49528125" y2="3.19535" width="0.1524" layer="1"/>
-<wire x1="40.63766875" y1="3.19535" x2="40.5478125" y2="3.206253125" width="0.1524" layer="1"/>
+<wire x1="100.4161875" y1="3.19535" x2="65.80156875" y2="3.19535" width="0.1524" layer="1"/>
+<wire x1="111.083121875" y1="13.862284375" x2="100.4161875" y2="3.19535" width="0.1524" layer="1"/>
+<wire x1="65.80156875" y1="3.19535" x2="65.01403125" y2="3.290909375" width="0.1524" layer="1"/>
+<wire x1="111.083121875" y1="24.783190625" x2="111.083121875" y2="13.862284375" width="0.1524" layer="1"/>
 </signal>
 <signal name="N$5">
@@
 <contactref element="BT1" pad="1"/>
 <wire x1="26.411325" y1="20.405803125" x2="35.55326875" y2="20.405803125" width="0.1524" layer="1"/>
-<wire x1="111.048215625" y1="44.7831625" x2="80.148996875" y2="13.88394375" width="0.1524" layer="1"/>
+<wire x1="111.048215625" y1="35.47075625" x2="89.461403125" y2="13.88394375" width="0.1524" layer="1"/>
 <wire x1="35.55326875" y1="20.405803125" x2="42.075128125" y2="13.88394375" width="0.1524" layer="1"/>
-<wire x1="42.075128125" y1="13.88394375" x2="80.148996875" y2="13.88394375" width="0.1524" layer="1"/>
+<wire x1="42.075128125" y1="13.88394375" x2="89.461403125" y2="13.88394375" width="0.1524" layer="1"/>
+<wire x1="111.048215625" y1="44.7831625" x2="111.048215625" y2="35.47075625" width="0.1524" layer="1"/>
 </signal>
 <signal name="N$4">
@@
 <contactref element="U1" pad="8"/>
 <contactref element="S1" pad="P"/>
-<wire x1="34.367546875" y1="6.85985625" x2="28.1036" y2="6.85985625" width="0.1524" layer="1"/>
-<wire x1="31.619646875" y1="3.343809375" x2="28.1036" y2="6.85985625" width="0.1524" layer="1"/>
+<wire x1="62.43446875" y1="3.343809375" x2="28.360496875" y2="3.343809375" width="0.1524" layer="1"/>
 <contactref element="R2" pad="P$2"/>
 <contactref element="R4" pad="P$2"/>
@@
 <contactref element="R3" pad="P$2"/>
 <wire x1="26.455496875" y1="3.343809375" x2="18.791325" y2="11.00798125" width="0.1524" layer="1"/>
-<wire x1="31.619646875" y1="3.343809375" x2="28.360496875" y2="3.343809375" width="0.1524" layer="1"/>
 <wire x1="28.360496875" y1="3.343809375" x2="28.23331875" y2="3.343809375" width="0.1524" layer="1"/>
 <wire x1="24.0007875" y1="3.343809375" x2="6.687996875" y2="20.6566" width="0.1524" layer="1"/>
@@
 <wire x1="19.132753125" y1="63.49403125" x2="19.132753125" y2="73.144684375" width="0.1524" layer="1"/>
 <wire x1="19.132753125" y1="73.144684375" x2="19.2174125" y2="73.22934375" width="0.1524" layer="1"/>
-<wire x1="38.00785" y1="3.219553125" x2="34.367546875" y2="6.85985625" width="0.1524" layer="1"/>
+<wire x1="62.47406875" y1="3.304209375" x2="62.43446875" y2="3.343809375" width="0.1524" layer="1"/>
 <wire x1="26.455496875" y1="3.343809375" x2="26.413359375" y2="3.343809375" width="0.1524" layer="1"/>
 <wire x1="26.413359375" y1="3.343809375" x2="24.97416875" y2="3.343809375" width="0.1524" layer="1"/>

Commit message: char badge
Routing:
- net N$6: track 205.0 -> 214.5 mm
- net N$4: track 65.2 -> 61.0 mm
Changed lines of the file:
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@@
 <contactref element="LED3" pad="K"/>
 <contactref element="LED4" pad="K"/>
-<wire x1="18.791325" y1="20.405803125" x2="12.52940625" y2="26.667721875" width="0.1524" layer="1"/>
-<wire x1="12.52940625" y1="26.667721875" x2="12.52940625" y2="43.5141875" width="0.1524" layer="1"/>
-<wire x1="18.791325" y1="20.405803125" x2="8.97376875" y2="30.223359375" width="0.1524" layer="1"/>
-<wire x1="8.97376875" y1="30.223359375" x2="8.97376875" y2="46.562009375" width="0.1524" layer="1"/>
-<wire x1="8.97376875" y1="46.562009375" x2="12.44464375" y2="50.032884375" width="0.1524" layer="1"/>
-<wire x1="16.846978125" y1="50.032884375" x2="12.44464375" y2="50.032884375" width="0.1524" layer="1"/>
+<wire x1="17.690765625" y1="20.405803125" x2="12.6142625" y2="25.48230625" width="0.1524" layer="1"/>
+<wire x1="12.6142625" y1="26.582865625" x2="12.6142625" y2="43.42933125" width="0.1524" layer="1"/>
+<wire x1="8.739334375" y1="47.68210625" x2="8.739334375" y2="29.27258125" width="0.1524" layer="1"/>
+<wire x1="8.739334375" y1="47.68210625" x2="11.0901125" y2="50.032884375" width="0.1524" layer="1"/>
+<wire x1="16.846978125" y1="50.032884375" x2="11.0901125" y2="50.032884375" width="0.1524" layer="1"/>
+<wire x1="18.791325" y1="20.405803125" x2="18.283375" y2="20.405803125" width="0.1524" layer="1"/>
+<wire x1="8.739334375" y1="29.27258125" x2="12.6142625" y2="25.397653125" width="0.1524" layer="1"/>
+<wire x1="18.791325" y1="20.405803125" x2="17.690765625" y2="20.405803125" width="0.1524" layer="1"/>
+<wire x1="12.6142625" y1="25.48230625" x2="12.6142625" y2="26.582865625" width="0.1524" layer="1"/>
+<wire x1="12.6142625" y1="43.42933125" x2="12.52940625" y2="43.5141875" width="0.1524" layer="1"/>
+<wire x1="12.6142625" y1="25.397653125" x2="12.6142625" y2="26.582865625" width="0.1524" layer="1"/>
 </signal>
 <signal name="N$6">
@@
 <wire x1="28.360496875" y1="3.343809375" x2="28.23331875" y2="3.343809375" width="0.1524" layer="1"/>
 <wire x1="24.0007875" y1="3.343809375" x2="6.687996875" y2="20.6566" width="0.1524" layer="1"/>
-<wire x1="6.687996875" y1="20.6566" x2="6.687996875" y2="42.498415625" width="0.1524" layer="1"/>
-<wire x1="6.687996875" y1="42.498415625" x2="6.687996875" y2="42.66773125" width="0.1524" layer="1"/>
+<wire x1="6.687996875" y1="34.625203125" x2="6.687996875" y2="40.72059375" width="0.1524" layer="1"/>
+<wire x1="6.687996875" y1="40.72059375" x2="6.687996875" y2="42.66773125" width="0.1524" layer="1"/>
 <wire x1="6.687996875" y1="42.66773125" x2="6.687996875" y2="51.641121875" width="0.1524" layer="1"/>
 <wire x1="6.687996875" y1="42.66773125" x2="6.687996875" y2="42.66773125" width="0.1524" layer="1"/>
-<wire x1="6.687996875" y1="42.498415625" x2="2.793721875" y2="46.392690625" width="0.1524" layer="1"/>
-<wire x1="2.793721875" y1="46.392690625" x2="2.793721875" y2="62.477753125" width="0.1524" layer="1"/>
-<wire x1="2.793721875" y1="62.477753125" x2="2.878378125" y2="62.477753125" width="0.1524" layer="1"/>
-<wire x1="2.878378125" y1="62.477753125" x2="8.405884375" y2="62.477753125" width="0.1524" layer="1"/>
-<wire x1="8.405884375" y1="62.477753125" x2="8.490628125" y2="62.562496875" width="0.1524" layer="1"/>
-<wire x1="2.878378125" y1="62.477753125" x2="2.878378125" y2="62.477753125" width="0.1524" layer="1"/>
-<wire x1="6.18005" y1="65.779425" x2="6.18005" y2="73.22934375" width="0.1524" layer="1"/>
-<wire x1="6.18005" y1="73.22934375" x2="19.2174125" y2="73.22934375" width="0.1524" layer="1"/>
-<wire x1="19.2174125" y1="73.22934375" x2="29.207084375" y2="73.22934375" width="0.1524" layer="1"/>
-<wire x1="22.434425" y1="66.456684375" x2="29.207084375" y2="73.22934375" width="0.1524" layer="1"/>
-<wire x1="22.434425" y1="66.456684375" x2="22.434425" y2="50.118034375" width="0.1524" layer="1"/>
-<wire x1="19.132753125" y1="63.49403125" x2="19.132753125" y2="73.144684375" width="0.1524" layer="1"/>
-<wire x1="19.132753125" y1="73.144684375" x2="19.2174125" y2="73.22934375" width="0.1524" layer="1"/>
+<wire x1="6.687996875" y1="34.625203125" x2="0" y2="41.3132" width="0.1524" layer="1"/>
+<wire x1="0" y1="41.3132" x2="0" y2="60.530615625" width="0.1524" layer="1"/>
+<wire x1="2.878378125" y1="63.40899375" x2="7.64413125" y2="63.40899375" width="0.1524" layer="1"/>
+<wire x1="3.386328125" y1="63.91694375" x2="3.386328125" y2="72.975365625" width="0.1524" layer="1"/>
+<wire x1="3.386328125" y1="72.975365625" x2="19.132753125" y2="72.975365625" width="0.1524" layer="1"/>
+<wire x1="20.487284375" y1="74.329896875" x2="26.602828125" y2="74.329896875" width="0.1524" layer="1"/>
+<wire x1="22.51908125" y1="70.24615" x2="26.602828125" y2="74.329896875" width="0.1524" layer="1"/>
+<wire x1="22.51908125" y1="70.24615" x2="22.51908125" y2="50.033378125" width="0.1524" layer="1"/>
 <wire x1="62.47406875" y1="3.304209375" x2="62.43446875" y2="3.343809375" width="0.1524" layer="1"/>
 <wire x1="26.455496875" y1="3.343809375" x2="26.413359375" y2="3.343809375" width="0.1524" layer="1"/>
@@
 <wire x1="18.791325" y1="11.00798125" x2="18.791325" y2="12.785803125" width="0.1524" layer="1"/>
 <wire x1="28.360496875" y1="3.343809375" x2="26.413359375" y2="3.343809375" width="0.1524" layer="1"/>
-<wire x1="2.878378125" y1="62.477753125" x2="6.18005" y2="65.779425" width="0.1524" layer="1"/>
-<wire x1="22.434425" y1="50.118034375" x2="22.51908125" y2="50.033378125" width="0.1524" layer="1"/>
+<wire x1="2.878378125" y1="63.40899375" x2="3.386328125" y2="63.91694375" width="0.1524" layer="1"/>
 <wire x1="24.97416875" y1="3.343809375" x2="24.0007875" y2="3.343809375" width="0.1524" layer="1"/>
+<wire x1="6.687996875" y1="20.6566" x2="6.687996875" y2="34.625203125" width="0.1524" layer="1"/>
+<wire x1="7.64413125" y1="63.40899375" x2="8.490628125" y2="62.562496875" width="0.1524" layer="1"/>
+<wire x1="0" y1="60.530615625" x2="2.878378125" y2="63.40899375" width="0.1524" layer="1"/>
+<wire x1="19.132753125" y1="72.975365625" x2="20.487284375" y2="74.329896875" width="0.1524" layer="1"/>
+<wire x1="19.132753125" y1="63.49403125" x2="19.132753125" y2="72.975365625" width="0.1524" layer="1"/>
 </signal>
 <signal name="N$1">
@@
 <contactref element="LED1" pad="K"/>
 <contactref element="LED2" pad="K"/>
-<wire x1="18.791325" y1="17.865803125" x2="7.703896875" y2="28.95323125" width="0.1524" layer="1"/>
-<wire x1="7.703896875" y1="28.95323125" x2="7.703896875" y2="48.424490625" width="0.1524" layer="1"/>
-<wire x1="7.703896875" y1="48.424490625" x2="11.80981875" y2="52.5304125" width="0.1524" layer="1"/>
+<wire x1="18.791325" y1="17.865803125" x2="7.788553125" y2="28.868575" width="0.1524" layer="1"/>
+<wire x1="7.788553125" y1="28.868575" x2="7.788553125" y2="48.509146875" width="0.1524" layer="1"/>
+<wire x1="7.788553125" y1="48.509146875" x2="11.80981875" y2="52.5304125" width="0.1524" layer="1"/>
 <wire x1="11.80981875" y1="52.5304125" x2="11.852146875" y2="52.572740625" width="0.1524" layer="1"/>
 <wire x1="11.852146875" y1="56.71645" x2="11.856575" y2="56.720878125" width="0.1524" layer="1"/>
@@
 </signal>
 <signal name="N$11">
-<via x="66.033396875" y="128.426490625" extent="1-16" drill="1"/>
+<via x="65.610103125" y="128.680465625" extent="1-16" drill="1"/>
 </signal>
 </signals>
