File: charbadge/charLED4inchess.brd (EAGLE design)
At the start: 79.4 x 79.4 mm, 6 parts, among them U1 ATTINY85-20P

Commit message: char badge
Routing:
- net N$1: track 105.2 -> 101.9 mm
Changed lines of the file:
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@@
 <contactref element="LED1" pad="K"/>
 <contactref element="LED2" pad="K"/>
-<wire x1="9.39325" y1="36.659540625" x2="3.851315625" y2="42.201475" width="0.1524" layer="1"/>
-<wire x1="3.851315625" y1="42.201475" x2="3.80961875" y2="42.243171875" width="0.1524" layer="1"/>
-<wire x1="3.80961875" y1="42.243171875" x2="3.80961875" y2="56.3823625" width="0.1524" layer="1"/>
-<wire x1="3.80961875" y1="56.3823625" x2="10.074325" y2="62.64706875" width="0.1524" layer="1"/>
+<wire x1="9.39325" y1="36.659540625" x2="5.29050625" y2="40.762284375" width="0.1524" layer="1"/>
+<wire x1="5.29050625" y1="40.762284375" x2="5.29050625" y2="57.25040625" width="0.1524" layer="1"/>
+<wire x1="5.29050625" y1="57.25040625" x2="10.074325" y2="62.034225" width="0.1524" layer="1"/>
 <wire x1="10.074325" y1="65.4407875" x2="15.831084375" y2="71.197546875" width="0.1524" layer="1"/>
 <wire x1="48.59380625" y1="71.197546875" x2="48.59380625" y2="59.853346875" width="0.1524" layer="1"/>
 <wire x1="48.59380625" y1="59.853346875" x2="48.5645125" y2="59.882640625" width="0.1524" layer="1"/>
 <wire x1="48.5645125" y1="59.882640625" x2="45.46819375" y2="59.882640625" width="0.1524" layer="1"/>
-<wire x1="10.074325" y1="62.64706875" x2="10.074325" y2="65.4407875" width="0.1524" layer="1"/>
+<wire x1="10.074325" y1="62.034225" x2="10.074325" y2="65.4407875" width="0.1524" layer="1"/>
 <wire x1="15.831084375" y1="71.197546875" x2="48.59380625" y2="71.197546875" width="0.1524" layer="1"/>
-<wire x1="8.379003125" y1="27.9407625" x2="3.851315625" y2="32.46845" width="0.1524" layer="1"/>
-<wire x1="3.851315625" y1="32.46845" x2="3.851315625" y2="42.201475" width="0.1524" layer="1"/>
+<wire x1="8.379003125" y1="27.9407625" x2="5.29050625" y2="31.029259375" width="0.1524" layer="1"/>
+<wire x1="5.29050625" y1="31.029259375" x2="5.29050625" y2="40.762284375" width="0.1524" layer="1"/>
 </signal>
 <signal name="N$2">
