File: astroCACTUS.brd (EAGLE design)
At the start: 160 x 100 mm, 13 parts, among them U1 ATTINY85-20P

Commit message: astro boy
Parts:
- added D11, D12, D13, D14, D15, D16, D17, D18: (no value), SparkFun-LED:LED_3MM
- moved D10 52.3 mm to (-99.1, -48.3)
- moved D9 52.3 mm to (-104.1, -48.3)
- moved D7 48.2 mm to (-104.1, -41.9)
- moved D8 46.0 mm to (-99.1, -41.9)
Connections:
- new net N$3: D11.K, D12.K, D13.K, D14.K, D15.K, D16.K, U1.7
- new net N$4: D10.K, D7.K, D8.K, D9.K, U1.6
- new net N$6: D17.K, D18.K, U1.5
- net N$1: now also D5.K, D6.K
- net N$31: now also D11.A, D17.A; no longer D10.A, D8.A, D9.A
Changed lines of the file:
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@@
 <attribute name="PROD_ID" value="DIO-08794" x="-83.82" y="3.81" size="1.778" layer="27" display="off"/>
 </element>
-<element name="D7" library="SparkFun-LED" library_urn="urn:adsk.eagle:library:529" package="LED_3MM" package3d_urn="urn:adsk.eagle:package:39361/1" value="" x="-88.9" y="3.81">
-<attribute name="PROD_ID" value="DIO-08794" x="-88.9" y="3.81" size="1.778" layer="27" display="off"/>
+<element name="D11" library="SparkFun-LED" library_urn="urn:adsk.eagle:library:529" package="LED_3MM" package3d_urn="urn:adsk.eagle:package:39361/1" value="" x="-104.14" y="-3.81">
+<attribute name="PROD_ID" value="DIO-08794" x="-109.22" y="3.81" size="1.778" layer="27" display="off"/>
 </element>
-<element name="D8" library="SparkFun-LED" library_urn="urn:adsk.eagle:library:529" package="LED_3MM" package3d_urn="urn:adsk.eagle:package:39361/1" value="" x="-93.98" y="3.81">
-<attribute name="PROD_ID" value="DIO-08794" x="-93.98" y="3.81" size="1.778" layer="27" display="off"/>
+<element name="D12" library="SparkFun-LED" library_urn="urn:adsk.eagle:library:529" package="LED_3MM" package3d_urn="urn:adsk.eagle:package:39361/1" value="" x="-104.14" y="-10.16">
+<attribute name="PROD_ID" value="DIO-08794" x="-109.22" y="-2.54" size="1.778" layer="27" display="off"/>
 </element>
-<element name="D9" library="SparkFun-LED" library_urn="urn:adsk.eagle:library:529" package="LED_3MM" package3d_urn="urn:adsk.eagle:package:39361/1" value="" x="-99.06" y="3.81">
-<attribute name="PROD_ID" value="DIO-08794" x="-99.06" y="3.81" size="1.778" layer="27" display="off"/>
+<element name="D13" library="SparkFun-LED" library_urn="urn:adsk.eagle:library:529" package="LED_3MM" package3d_urn="urn:adsk.eagle:package:39361/1" value="" x="-104.14" y="-16.51">
+<attribute name="PROD_ID" value="DIO-08794" x="-109.22" y="-8.89" size="1.778" layer="27" display="off"/>
 </element>
-<element name="D10" library="SparkFun-LED" library_urn="urn:adsk.eagle:library:529" package="LED_3MM" package3d_urn="urn:adsk.eagle:package:39361/1" value="" x="-104.14" y="3.81">
-<attribute name="PROD_ID" value="DIO-08794" x="-104.14" y="3.81" size="1.778" layer="27" display="off"/>
+<element name="D14" library="SparkFun-LED" library_urn="urn:adsk.eagle:library:529" package="LED_3MM" package3d_urn="urn:adsk.eagle:package:39361/1" value="" x="-104.14" y="-22.86">
+<attribute name="PROD_ID" value="DIO-08794" x="-109.22" y="-15.24" size="1.778" layer="27" display="off"/>
+</element>
+<element name="D15" library="SparkFun-LED" library_urn="urn:adsk.eagle:library:529" package="LED_3MM" package3d_urn="urn:adsk.eagle:package:39361/1" value="" x="-104.14" y="-29.21">
+<attribute name="PROD_ID" value="DIO-08794" x="-109.22" y="-21.59" size="1.778" layer="27" display="off"/>
+</element>
+<element name="D16" library="SparkFun-LED" library_urn="urn:adsk.eagle:library:529" package="LED_3MM" package3d_urn="urn:adsk.eagle:package:39361/1" value="" x="-104.14" y="-35.56">
+<attribute name="PROD_ID" value="DIO-08794" x="-109.22" y="-27.94" size="1.778" layer="27" display="off"/>
+</element>
+<element name="D7" library="SparkFun-LED" library_urn="urn:adsk.eagle:library:529" package="LED_3MM" package3d_urn="urn:adsk.eagle:package:39361/1" value="" x="-104.14" y="-41.91">
+<attribute name="PROD_ID" value="DIO-08794" x="-109.22" y="-34.29" size="1.778" layer="27" display="off"/>
+</element>
+<element name="D8" library="SparkFun-LED" library_urn="urn:adsk.eagle:library:529" package="LED_3MM" package3d_urn="urn:adsk.eagle:package:39361/1" value="" x="-99.06" y="-41.91">
+<attribute name="PROD_ID" value="DIO-08794" x="-114.3" y="-34.29" size="1.778" layer="27" display="off"/>
+</element>
+<element name="D9" library="SparkFun-LED" library_urn="urn:adsk.eagle:library:529" package="LED_3MM" package3d_urn="urn:adsk.eagle:package:39361/1" value="" x="-104.14" y="-48.26">
+<attribute name="PROD_ID" value="DIO-08794" x="-119.38" y="-34.29" size="1.778" layer="27" display="off"/>
+</element>
+<element name="D10" library="SparkFun-LED" library_urn="urn:adsk.eagle:library:529" package="LED_3MM" package3d_urn="urn:adsk.eagle:package:39361/1" value="" x="-99.06" y="-48.26">
+<attribute name="PROD_ID" value="DIO-08794" x="-124.46" y="-34.29" size="1.778" layer="27" display="off"/>
+</element>
+<element name="D17" library="SparkFun-LED" library_urn="urn:adsk.eagle:library:529" package="LED_3MM" package3d_urn="urn:adsk.eagle:package:39361/1" value="" x="-104.14" y="-54.61">
+<attribute name="PROD_ID" value="DIO-08794" x="-109.22" y="-46.99" size="1.778" layer="27" display="off"/>
+</element>
+<element name="D18" library="SparkFun-LED" library_urn="urn:adsk.eagle:library:529" package="LED_3MM" package3d_urn="urn:adsk.eagle:package:39361/1" value="" x="-104.14" y="-60.96">
+<attribute name="PROD_ID" value="DIO-08794" x="-114.3" y="-46.99" size="1.778" layer="27" display="off"/>
 </element>
 </elements>
@@
 <contactref element="U1" pad="8"/>
 <contactref element="S1" pad="P"/>
-<contactref element="D10" pad="A"/>
-<contactref element="D9" pad="A"/>
-<contactref element="D8" pad="A"/>
-<contactref element="D7" pad="A"/>
 <contactref element="D6" pad="A"/>
 <contactref element="D5" pad="A"/>
@@
 <contactref element="D2" pad="A"/>
 <contactref element="D1" pad="A"/>
-<wire x1="-100.33" y1="3.81" x2="-105.41" y2="3.81" width="0" layer="19" extent="1-1"/>
-<wire x1="-95.25" y1="3.81" x2="-100.33" y2="3.81" width="0" layer="19" extent="1-1"/>
-<wire x1="-90.17" y1="3.81" x2="-95.25" y2="3.81" width="0" layer="19" extent="1-1"/>
-<wire x1="-85.09" y1="3.81" x2="-90.17" y2="3.81" width="0" layer="19" extent="1-1"/>
+<contactref element="D11" pad="A"/>
+<contactref element="D7" pad="A"/>
+<contactref element="D17" pad="A"/>
+<wire x1="-105.41" y1="-41.91" x2="-105.41" y2="-54.61" width="0" layer="19" extent="1-1"/>
+<wire x1="-105.41" y1="-3.81" x2="-105.41" y2="-41.91" width="0" layer="19" extent="1-1"/>
+<wire x1="-85.09" y1="3.81" x2="-105.41" y2="-3.81" width="0" layer="19" extent="1-1"/>
 <wire x1="-80.01" y1="3.81" x2="-85.09" y2="3.81" width="0" layer="19" extent="1-1"/>
 <wire x1="-74.93" y1="3.81" x2="-80.01" y2="3.81" width="0" layer="19" extent="1-1"/>
@@
 <contactref element="D3" pad="K"/>
 <contactref element="D4" pad="K"/>
+<contactref element="D5" pad="K"/>
+<contactref element="D6" pad="K"/>
+<wire x1="-77.47" y1="3.81" x2="-82.55" y2="3.81" width="0" layer="19" extent="1-1"/>
+<wire x1="-72.39" y1="3.81" x2="-77.47" y2="3.81" width="0" layer="19" extent="1-1"/>
 <wire x1="-67.31" y1="3.81" x2="-72.39" y2="3.81" width="0" layer="19" extent="1-1"/>
 <wire x1="-62.23" y1="3.81" x2="-67.31" y2="3.81" width="0" layer="19" extent="1-1"/>
@@
 <wire x1="-50.8" y1="2.54" x2="-57.15" y2="3.81" width="0" layer="19" extent="1-1"/>
 </signal>
+<signal name="N$3">
+<contactref element="U1" pad="7"/>
+<contactref element="D11" pad="K"/>
+<contactref element="D12" pad="K"/>
+<contactref element="D13" pad="K"/>
+<contactref element="D14" pad="K"/>
+<contactref element="D15" pad="K"/>
+<contactref element="D16" pad="K"/>
+<wire x1="-102.87" y1="-29.21" x2="-102.87" y2="-35.56" width="0" layer="19" extent="1-1"/>
+<wire x1="-102.87" y1="-22.86" x2="-102.87" y2="-29.21" width="0" layer="19" extent="1-1"/>
+<wire x1="-102.87" y1="-16.51" x2="-102.87" y2="-22.86" width="0" layer="19" extent="1-1"/>
+<wire x1="-102.87" y1="-10.16" x2="-102.87" y2="-16.51" width="0" layer="19" extent="1-1"/>
+<wire x1="-102.87" y1="-3.81" x2="-102.87" y2="-10.16" width="0" layer="19" extent="1-1"/>
+<wire x1="-50.8" y1="10.16" x2="-102.87" y2="-3.81" width="0" layer="19" extent="1-1"/>
+</signal>
+<signal name="N$4">
+<contactref element="U1" pad="6"/>
+<contactref element="D7" pad="K"/>
+<contactref element="D8" pad="K"/>
+<contactref element="D9" pad="K"/>
+<contactref element="D10" pad="K"/>
+<wire x1="-97.79" y1="-48.26" x2="-102.87" y2="-48.26" width="0" layer="19" extent="1-1"/>
+<wire x1="-102.87" y1="-41.91" x2="-102.87" y2="-48.26" width="0" layer="19" extent="1-1"/>
+<wire x1="-97.79" y1="-41.91" x2="-102.87" y2="-41.91" width="0" layer="19" extent="1-1"/>
+<wire x1="-48.26" y1="10.16" x2="-97.79" y2="-41.91" width="0" layer="19" extent="1-1"/>
+</signal>
+<signal name="N$6">
+<contactref element="U1" pad="5"/>
+<contactref element="D17" pad="K"/>
+<contactref element="D18" pad="K"/>
+<wire x1="-102.87" y1="-54.61" x2="-102.87" y2="-60.96" width="0" layer="19" extent="1-1"/>
+<wire x1="-45.72" y1="10.16" x2="-102.87" y2="-54.61" width="0" layer="19" extent="1-1"/>
+</signal>
 </signals>

Commit message: astro boy
Parts:
- moved D18 153.8 mm to (27.8, 18.0), turned to 92.5 degrees
- moved D9 151.3 mm to (32.8, 16.1), turned to 90.7 degrees
- moved D17 142.4 mm to (22.3, 10.7), turned to 92.4 degrees
- moved D8 138.2 mm to (27.9, 12.7), turned to 90.6 degrees
- moved D7 134.9 mm to (22.4, 4.74), turned to 91.8 degrees
- moved D10 129.2 mm to (17.3, 7.87), turned to 91.7 degrees
Other:
- board outline removed
- board text added: "/Users/chrisbuckner/badges/fresh/astro_copper_only.bmp"
- board text added: "/Users/chrisbuckner/badges/fresh/astro_silk_only_no_fire_bitmap.bmp"

Commit message: astro boy
Parts:
- moved D14 142.5 mm to (34.7, 9.39), turned to 92.1 degrees
- moved D15 136.7 mm to (27.9, 6.01), turned to 93 degrees
- moved D16 132.7 mm to (25.4, -6.61), turned to 90.5 degrees
- moved D13 132.3 mm to (27.2, -0.17), turned to 91.2 degrees
- moved D12 126.0 mm to (21.7, -2.71), turned to 87.5 degrees
- moved D11 118.7 mm to (14.4, 1.86), turned to 87.5 degrees
- moved D6 117.3 mm to (33.4, 1.86), turned to 90 degrees
- moved D5 109.8 mm to (30.7, -4.15), turned to 90 degrees
- moved D3 98.4 mm to (28.6, -11.5), turned to 90 degrees
- moved D4 95.6 mm to (20.8, -10.7), turned to 90.7 degrees
- moved D2 89.3 mm to (22.9, -18.5), turned to 90.4 degrees
- moved D1 75.4 mm to (16.4, -5.08), turned to 89.5 degrees
- moved D8 1.57 mm to (29.2, 11.8)
- moved D7 1.27 mm to (21.4, 3.97)
- moved D10 0.92 mm to (16.6, 8.38)
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
Commit message: astro boy
Parts:
- moved D2 1.26 mm to (23.8, -17.6)
Changed lines of the file:
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@@
 <attribute name="PROD_ID" value="DIO-08794" x="16.41785" y="-5.0791125" size="1.778" layer="27" rot="R89.5" display="off"/>
 </element>
-<element name="D2" library="SparkFun-LED" library_urn="urn:adsk.eagle:library:529" package="LED_3MM" package3d_urn="urn:adsk.eagle:package:39361/1" value="" x="22.936025" y="-18.539765625" rot="R90.4">
-<attribute name="PROD_ID" value="DIO-08794" x="22.936025" y="-18.539765625" size="1.778" layer="27" rot="R90.4" display="off"/>
+<element name="D2" library="SparkFun-LED" library_urn="urn:adsk.eagle:library:529" package="LED_3MM" package3d_urn="urn:adsk.eagle:package:39361/1" value="" x="23.782609375" y="-17.608525" rot="R90.4">
+<attribute name="PROD_ID" value="DIO-08794" x="23.782609375" y="-17.608525" size="1.778" layer="27" rot="R90.4" display="off"/>
 </element>
 <element name="D3" library="SparkFun-LED" library_urn="urn:adsk.eagle:library:529" package="LED_3MM" package3d_urn="urn:adsk.eagle:package:39361/1" value="" x="28.607609375" y="-11.513140625" rot="R90">
@@
 <wire x1="20.8340625" y1="-11.936453125" x2="30.72305625" y2="-5.41786875" width="0" layer="19" extent="1-1"/>
 <wire x1="28.607609375" y1="-12.783140625" x2="20.8340625" y2="-11.936453125" width="0" layer="19" extent="1-1"/>
-<wire x1="22.944890625" y1="-19.809734375" x2="28.607609375" y2="-12.783140625" width="0" layer="19" extent="1-1"/>
-<wire x1="16.406765625" y1="-6.3490625" x2="22.944890625" y2="-19.809734375" width="0" layer="19" extent="1-1"/>
+<wire x1="23.791475" y1="-18.87849375" x2="28.607609375" y2="-12.783140625" width="0" layer="19" extent="1-1"/>
+<wire x1="16.406765625" y1="-6.3490625" x2="23.791475" y2="-18.87849375" width="0" layer="19" extent="1-1"/>
 <wire x1="-53.34" y1="10.16" x2="16.406765625" y2="-6.3490625" width="0" layer="19" extent="1-1"/>
 <wire x1="-44.45" y1="48.26" x2="-53.34" y2="10.16" width="0" layer="19" extent="1-1"/>
@@
 <wire x1="20.803034375" y1="-9.39664375" x2="30.72305625" y2="-2.87786875" width="0" layer="19" extent="1-1"/>
 <wire x1="28.607609375" y1="-10.243140625" x2="20.803034375" y2="-9.39664375" width="0" layer="19" extent="1-1"/>
-<wire x1="22.92715625" y1="-17.26979375" x2="28.607609375" y2="-10.243140625" width="0" layer="19" extent="1-1"/>
-<wire x1="16.42893125" y1="-3.809159375" x2="22.92715625" y2="-17.26979375" width="0" layer="19" extent="1-1"/>
+<wire x1="23.773740625" y1="-16.338553125" x2="28.607609375" y2="-10.243140625" width="0" layer="19" extent="1-1"/>
+<wire x1="16.42893125" y1="-3.809159375" x2="23.773740625" y2="-16.338553125" width="0" layer="19" extent="1-1"/>
 <wire x1="-50.8" y1="2.54" x2="16.42893125" y2="-3.809159375" width="0" layer="19" extent="1-1"/>
 </signal>

Commit message: astro boy
Parts:
- moved D2 1.26 mm to (22.9, -18.5)
- moved D6 0.19 mm to (33.5, 2.03)
Changed lines of the file:
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@@
 <attribute name="PROD_ID" value="DIO-08794" x="16.41785" y="-5.0791125" size="1.778" layer="27" rot="R89.5" display="off"/>
 </element>
-<element name="D2" library="SparkFun-LED" library_urn="urn:adsk.eagle:library:529" package="LED_3MM" package3d_urn="urn:adsk.eagle:package:39361/1" value="" x="23.782609375" y="-17.608525" rot="R90.4">
-<attribute name="PROD_ID" value="DIO-08794" x="23.782609375" y="-17.608525" size="1.778" layer="27" rot="R90.4" display="off"/>
+<element name="D2" library="SparkFun-LED" library_urn="urn:adsk.eagle:library:529" package="LED_3MM" package3d_urn="urn:adsk.eagle:package:39361/1" value="" x="22.936025" y="-18.539765625" rot="R90.4">
+<attribute name="PROD_ID" value="DIO-08794" x="22.936025" y="-18.539765625" size="1.778" layer="27" rot="R90.4" display="off"/>
 </element>
 <element name="D3" library="SparkFun-LED" library_urn="urn:adsk.eagle:library:529" package="LED_3MM" package3d_urn="urn:adsk.eagle:package:39361/1" value="" x="28.607609375" y="-11.513140625" rot="R90">
@@
 <attribute name="PROD_ID" value="DIO-08794" x="30.72305625" y="-4.14786875" size="1.778" layer="27" rot="R90" display="off"/>
 </element>
-<element name="D6" library="SparkFun-LED" library_urn="urn:adsk.eagle:library:529" package="LED_3MM" package3d_urn="urn:adsk.eagle:package:39361/1" value="" x="33.431609375" y="1.8628625" rot="R90">
-<attribute name="PROD_ID" value="DIO-08794" x="33.431609375" y="1.8628625" size="1.778" layer="27" rot="R90" display="off"/>
+<element name="D6" library="SparkFun-LED" library_urn="urn:adsk.eagle:library:529" package="LED_3MM" package3d_urn="urn:adsk.eagle:package:39361/1" value="" x="33.51626875" y="2.03218125" rot="R90">
+<attribute name="PROD_ID" value="DIO-08794" x="33.51626875" y="2.03218125" size="1.778" layer="27" rot="R90" display="off"/>
 </element>
 <element name="D11" library="SparkFun-LED" library_urn="urn:adsk.eagle:library:529" package="LED_3MM" package3d_urn="urn:adsk.eagle:package:39361/1" value="" x="14.3814875" y="1.862096875" rot="R87.5">
@@
 <wire x1="21.448003125" y1="2.705375" x2="22.477190625" y2="8.715321875" width="0" layer="19" extent="1-1"/>
 <wire x1="14.326090625" y1="0.59330625" x2="21.448003125" y2="2.705375" width="0" layer="19" extent="1-1"/>
-<wire x1="33.431609375" y1="0.5928625" x2="14.326090625" y2="0.59330625" width="0" layer="19" extent="1-1"/>
-<wire x1="30.72305625" y1="-5.41786875" x2="33.431609375" y2="0.5928625" width="0" layer="19" extent="1-1"/>
+<wire x1="33.51626875" y1="0.76218125" x2="14.326090625" y2="0.59330625" width="0" layer="19" extent="1-1"/>
+<wire x1="30.72305625" y1="-5.41786875" x2="33.51626875" y2="0.76218125" width="0" layer="19" extent="1-1"/>
 <wire x1="20.8340625" y1="-11.936453125" x2="30.72305625" y2="-5.41786875" width="0" layer="19" extent="1-1"/>
 <wire x1="28.607609375" y1="-12.783140625" x2="20.8340625" y2="-11.936453125" width="0" layer="19" extent="1-1"/>
-<wire x1="23.791475" y1="-18.87849375" x2="28.607609375" y2="-12.783140625" width="0" layer="19" extent="1-1"/>
-<wire x1="16.406765625" y1="-6.3490625" x2="23.791475" y2="-18.87849375" width="0" layer="19" extent="1-1"/>
+<wire x1="22.944890625" y1="-19.809734375" x2="28.607609375" y2="-12.783140625" width="0" layer="19" extent="1-1"/>
+<wire x1="16.406765625" y1="-6.3490625" x2="22.944890625" y2="-19.809734375" width="0" layer="19" extent="1-1"/>
 <wire x1="-53.34" y1="10.16" x2="16.406765625" y2="-6.3490625" width="0" layer="19" extent="1-1"/>
 <wire x1="-44.45" y1="48.26" x2="-53.34" y2="10.16" width="0" layer="19" extent="1-1"/>
@@
 <contactref element="D5" pad="K"/>
 <contactref element="D6" pad="K"/>
-<wire x1="30.72305625" y1="-2.87786875" x2="33.431609375" y2="3.1328625" width="0" layer="19" extent="1-1"/>
+<wire x1="30.72305625" y1="-2.87786875" x2="33.51626875" y2="3.30218125" width="0" layer="19" extent="1-1"/>
 <wire x1="20.803034375" y1="-9.39664375" x2="30.72305625" y2="-2.87786875" width="0" layer="19" extent="1-1"/>
 <wire x1="28.607609375" y1="-10.243140625" x2="20.803034375" y2="-9.39664375" width="0" layer="19" extent="1-1"/>
-<wire x1="23.773740625" y1="-16.338553125" x2="28.607609375" y2="-10.243140625" width="0" layer="19" extent="1-1"/>
-<wire x1="16.42893125" y1="-3.809159375" x2="23.773740625" y2="-16.338553125" width="0" layer="19" extent="1-1"/>
+<wire x1="22.92715625" y1="-17.26979375" x2="28.607609375" y2="-10.243140625" width="0" layer="19" extent="1-1"/>
+<wire x1="16.42893125" y1="-3.809159375" x2="22.92715625" y2="-17.26979375" width="0" layer="19" extent="1-1"/>
 <wire x1="-50.8" y1="2.54" x2="16.42893125" y2="-3.809159375" width="0" layer="19" extent="1-1"/>
 </signal>
