File: astroCACTUS.brd (EAGLE design)
At the start: 57.7 x 135.1 mm, 21 parts, among them U1 ATTINY85-20P

Commit message: astro boy
Parts:
- moved D15 1.71 mm to (28.5, 6.43)
- moved D1 1.61 mm to (16.4, -3.47)
- moved D4 1.18 mm to (20.1, -11.6)
- moved D8 0.77 mm to (26.9, 12.1)
- moved D12 0.59 mm to (21.7, -2.12)
- moved D11 0.51 mm to (13.9, 1.86)
- moved D14 0.51 mm to (34.5, 8.12)
- moved D10 0.51 mm to (17.1, 8.38)
- moved D17 0.43 mm to (22.0, 9.90)
- moved D5 0.34 mm to (30.8, -4.74)
- moved D16 0.25 mm to (25.4, -6.86)
- moved D7 0.12 mm to (20.7, 4.06)
- moved D18 0.12 mm to (29.2, 18.5)
- moved D9 0.12 mm to (32.7, 13.3)
Routing:
- net N$31: track 323.1 -> 338.6 mm
- net N$1: track 104.9 -> 104.1 mm
- net N$3: track 80.3 -> 79.7 mm
