File: astroCACTUS.sch (EAGLE design)
At the start: 13 parts, among them U1 ATTINY85-20P

Commit message: astro boy
Parts:
- added D11, D12, D13, D14, D15, D16, D17, D18: (no value), SparkFun-LED:LED3MM
Connections:
- new net N$3: D11.C, D12.C, D13.C, D14.C, D15.C, D16.C, U1.PB2
- new net N$4: D10.C, D7.C, D8.C, D9.C, U1.PB1
- new net N$6: D17.C, D18.C, U1.PB0
- net N$1: now also D5.C, D6.C
- net N$31: now also D11.A, D17.A; no longer D10.A, D8.A, D9.A
Other:
- moved on the sheet: D10, D7, D8, D9
Changed lines of the file:
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@@
 <part name="D5" library="SparkFun-LED" library_urn="urn:adsk.eagle:library:529" deviceset="LED" device="3MM" package3d_urn="urn:adsk.eagle:package:39361/1"/>
 <part name="D6" library="SparkFun-LED" library_urn="urn:adsk.eagle:library:529" deviceset="LED" device="3MM" package3d_urn="urn:adsk.eagle:package:39361/1"/>
+<part name="D11" library="SparkFun-LED" library_urn="urn:adsk.eagle:library:529" deviceset="LED" device="3MM" package3d_urn="urn:adsk.eagle:package:39361/1"/>
+<part name="D12" library="SparkFun-LED" library_urn="urn:adsk.eagle:library:529" deviceset="LED" device="3MM" package3d_urn="urn:adsk.eagle:package:39361/1"/>
+<part name="D13" library="SparkFun-LED" library_urn="urn:adsk.eagle:library:529" deviceset="LED" device="3MM" package3d_urn="urn:adsk.eagle:package:39361/1"/>
+<part name="D14" library="SparkFun-LED" library_urn="urn:adsk.eagle:library:529" deviceset="LED" device="3MM" package3d_urn="urn:adsk.eagle:package:39361/1"/>
+<part name="D15" library="SparkFun-LED" library_urn="urn:adsk.eagle:library:529" deviceset="LED" device="3MM" package3d_urn="urn:adsk.eagle:package:39361/1"/>
+<part name="D16" library="SparkFun-LED" library_urn="urn:adsk.eagle:library:529" deviceset="LED" device="3MM" package3d_urn="urn:adsk.eagle:package:39361/1"/>
 <part name="D7" library="SparkFun-LED" library_urn="urn:adsk.eagle:library:529" deviceset="LED" device="3MM" package3d_urn="urn:adsk.eagle:package:39361/1"/>
 <part name="D8" library="SparkFun-LED" library_urn="urn:adsk.eagle:library:529" deviceset="LED" device="3MM" package3d_urn="urn:adsk.eagle:package:39361/1"/>
 <part name="D9" library="SparkFun-LED" library_urn="urn:adsk.eagle:library:529" deviceset="LED" device="3MM" package3d_urn="urn:adsk.eagle:package:39361/1"/>
 <part name="D10" library="SparkFun-LED" library_urn="urn:adsk.eagle:library:529" deviceset="LED" device="3MM" package3d_urn="urn:adsk.eagle:package:39361/1"/>
+<part name="D17" library="SparkFun-LED" library_urn="urn:adsk.eagle:library:529" deviceset="LED" device="3MM" package3d_urn="urn:adsk.eagle:package:39361/1"/>
+<part name="D18" library="SparkFun-LED" library_urn="urn:adsk.eagle:library:529" deviceset="LED" device="3MM" package3d_urn="urn:adsk.eagle:package:39361/1"/>
 </parts>
 <sheets>
@@
 <instance part="D5" gate="G$1" x="121.92" y="71.12"/>
 <instance part="D6" gate="G$1" x="137.16" y="71.12"/>
-<instance part="D7" gate="G$1" x="149.86" y="71.12"/>
-<instance part="D8" gate="G$1" x="160.02" y="71.12"/>
-<instance part="D9" gate="G$1" x="172.72" y="71.12"/>
-<instance part="D10" gate="G$1" x="185.42" y="71.12"/>
+<instance part="D11" gate="G$1" x="63.5" y="50.8"/>
+<instance part="D12" gate="G$1" x="78.74" y="50.8"/>
+<instance part="D13" gate="G$1" x="93.98" y="50.8"/>
+<instance part="D14" gate="G$1" x="106.68" y="50.8"/>
+<instance part="D15" gate="G$1" x="121.92" y="50.8"/>
+<instance part="D16" gate="G$1" x="137.16" y="50.8"/>
+<instance part="D7" gate="G$1" x="63.5" y="33.02"/>
+<instance part="D8" gate="G$1" x="78.74" y="33.02"/>
+<instance part="D9" gate="G$1" x="93.98" y="33.02"/>
+<instance part="D10" gate="G$1" x="106.68" y="33.02"/>
+<instance part="D17" gate="G$1" x="63.5" y="17.78"/>
+<instance part="D18" gate="G$1" x="78.74" y="17.78"/>
 </instances>
 <busses>
@@
 <wire x1="-20.32" y1="76.2" x2="-20.32" y2="86.36" width="0.1524" layer="91"/>
 <junction x="-20.32" y="76.2"/>
-<pinref part="D10" gate="G$1" pin="A"/>
 <wire x1="-20.32" y1="86.36" x2="63.5" y2="86.36" width="0.1524" layer="91"/>
 <wire x1="63.5" y1="86.36" x2="78.74" y2="86.36" width="0.1524" layer="91"/>
@@
 <wire x1="106.68" y1="86.36" x2="121.92" y2="86.36" width="0.1524" layer="91"/>
 <wire x1="121.92" y1="86.36" x2="137.16" y2="86.36" width="0.1524" layer="91"/>
-<wire x1="137.16" y1="86.36" x2="149.86" y2="86.36" width="0.1524" layer="91"/>
-<wire x1="149.86" y1="86.36" x2="160.02" y2="86.36" width="0.1524" layer="91"/>
-<wire x1="160.02" y1="86.36" x2="172.72" y2="86.36" width="0.1524" layer="91"/>
-<wire x1="172.72" y1="86.36" x2="185.42" y2="86.36" width="0.1524" layer="91"/>
-<wire x1="185.42" y1="86.36" x2="185.42" y2="73.66" width="0.1524" layer="91"/>
-<pinref part="D9" gate="G$1" pin="A"/>
-<wire x1="172.72" y1="73.66" x2="172.72" y2="86.36" width="0.1524" layer="91"/>
-<junction x="172.72" y="86.36"/>
-<pinref part="D8" gate="G$1" pin="A"/>
-<wire x1="160.02" y1="73.66" x2="160.02" y2="86.36" width="0.1524" layer="91"/>
-<junction x="160.02" y="86.36"/>
-<pinref part="D7" gate="G$1" pin="A"/>
-<wire x1="149.86" y1="73.66" x2="149.86" y2="86.36" width="0.1524" layer="91"/>
-<junction x="149.86" y="86.36"/>
 <pinref part="D6" gate="G$1" pin="A"/>
 <wire x1="137.16" y1="73.66" x2="137.16" y2="86.36" width="0.1524" layer="91"/>
-<junction x="137.16" y="86.36"/>
 <pinref part="D5" gate="G$1" pin="A"/>
 <wire x1="121.92" y1="73.66" x2="121.92" y2="86.36" width="0.1524" layer="91"/>
@@
 <wire x1="63.5" y1="73.66" x2="63.5" y2="86.36" width="0.1524" layer="91"/>
 <junction x="63.5" y="86.36"/>
+<wire x1="137.16" y1="86.36" x2="144.78" y2="86.36" width="0.1524" layer="91"/>
+<wire x1="144.78" y1="86.36" x2="144.78" y2="53.34" width="0.1524" layer="91"/>
+<junction x="137.16" y="86.36"/>
+<pinref part="D11" gate="G$1" pin="A"/>
+<wire x1="144.78" y1="53.34" x2="63.5" y2="53.34" width="0.1524" layer="91"/>
+<pinref part="D7" gate="G$1" pin="A"/>
+<wire x1="144.78" y1="53.34" x2="144.78" y2="35.56" width="0.1524" layer="91"/>
+<wire x1="144.78" y1="35.56" x2="63.5" y2="35.56" width="0.1524" layer="91"/>
+<junction x="144.78" y="53.34"/>
+<wire x1="144.78" y1="35.56" x2="144.78" y2="20.32" width="0.1524" layer="91"/>
+<junction x="144.78" y="35.56"/>
+<pinref part="D17" gate="G$1" pin="A"/>
+<wire x1="144.78" y1="20.32" x2="63.5" y2="20.32" width="0.1524" layer="91"/>
 </segment>
 </net>
@@
 <wire x1="106.68" y1="63.5" x2="106.68" y2="66.04" width="0.1524" layer="91"/>
 <junction x="93.98" y="63.5"/>
-</segment>
-</net>
+<pinref part="D5" gate="G$1" pin="C"/>
+<wire x1="106.68" y1="63.5" x2="121.92" y2="63.5" width="0.1524" layer="91"/>
+<wire x1="121.92" y1="63.5" x2="121.92" y2="66.04" width="0.1524" layer="91"/>
+<junction x="106.68" y="63.5"/>
+<pinref part="D6" gate="G$1" pin="C"/>
+<wire x1="121.92" y1="63.5" x2="137.16" y2="63.5" width="0.1524" layer="91"/>
+<wire x1="137.16" y1="63.5" x2="137.16" y2="66.04" width="0.1524" layer="91"/>
+<junction x="121.92" y="63.5"/>
+</segment>
+</net>
+<net name="N$3" class="0">
+<segment>
+<pinref part="U1" gate="G$1" pin="PB2"/>
+<wire x1="33.02" y1="68.58" x2="53.34" y2="68.58" width="0.1524" layer="91"/>
+<wire x1="53.34" y1="68.58" x2="53.34" y2="43.18" width="0.1524" layer="91"/>
+<pinref part="D11" gate="G$1" pin="C"/>
+<wire x1="53.34" y1="43.18" x2="63.5" y2="43.18" width="0.1524" layer="91"/>
+<wire x1="63.5" y1="43.18" x2="63.5" y2="45.72" width="0.1524" layer="91"/>
+<pinref part="D12" gate="G$1" pin="C"/>
+<wire x1="63.5" y1="43.18" x2="78.74" y2="43.18" width="0.1524" layer="91"/>
+<wire x1="78.74" y1="43.18" x2="78.74" y2="45.72" width="0.1524" layer="91"/>
+<junction x="63.5" y="43.18"/>
+<pinref part="D13" gate="G$1" pin="C"/>
+<wire x1="78.74" y1="43.18" x2="93.98" y2="43.18" width="0.1524" layer="91"/>
+<wire x1="93.98" y1="43.18" x2="93.98" y2="45.72" width="0.1524" layer="91"/>
+<junction x="78.74" y="43.18"/>
+<pinref part="D14" gate="G$1" pin="C"/>
+<wire x1="93.98" y1="43.18" x2="106.68" y2="43.18" width="0.1524" layer="91"/>
+<wire x1="106.68" y1="43.18" x2="106.68" y2="45.72" width="0.1524" layer="91"/>
+<junction x="93.98" y="43.18"/>
+<pinref part="D15" gate="G$1" pin="C"/>
+<wire x1="106.68" y1="43.18" x2="121.92" y2="43.18" width="0.1524" layer="91"/>
+<wire x1="121.92" y1="43.18" x2="121.92" y2="45.72" width="0.1524" layer="91"/>
+<junction x="106.68" y="43.18"/>
+<pinref part="D16" gate="G$1" pin="C"/>
+<wire x1="121.92" y1="43.18" x2="137.16" y2="43.18" width="0.1524" layer="91"/>
+<wire x1="137.16" y1="43.18" x2="137.16" y2="45.72" width="0.1524" layer="91"/>
+<junction x="121.92" y="43.18"/>
+</segment>
+</net>
+<net name="N$4" class="0">
+<segment>
+<pinref part="U1" gate="G$1" pin="PB1"/>
+<wire x1="33.02" y1="66.04" x2="50.8" y2="66.04" width="0.1524" layer="91"/>
+<wire x1="50.8" y1="66.04" x2="50.8" y2="25.4" width="0.1524" layer="91"/>
+<pinref part="D7" gate="G$1" pin="C"/>
+<wire x1="50.8" y1="25.4" x2="63.5" y2="25.4" width="0.1524" layer="91"/>
+<wire x1="63.5" y1="25.4" x2="63.5" y2="27.94" width="0.1524" layer="91"/>
+<pinref part="D8" gate="G$1" pin="C"/>
+<wire x1="63.5" y1="25.4" x2="78.74" y2="25.4" width="0.1524" layer="91"/>
+<wire x1="78.74" y1="25.4" x2="78.74" y2="27.94" width="0.1524" layer="91"/>
+<junction x="63.5" y="25.4"/>
+<pinref part="D9" gate="G$1" pin="C"/>
+<wire x1="78.74" y1="25.4" x2="93.98" y2="25.4" width="0.1524" layer="91"/>
+<wire x1="93.98" y1="25.4" x2="93.98" y2="27.94" width="0.1524" layer="91"/>
+<junction x="78.74" y="25.4"/>
+<pinref part="D10" gate="G$1" pin="C"/>
+<wire x1="93.98" y1="25.4" x2="106.68" y2="25.4" width="0.1524" layer="91"/>
+<wire x1="106.68" y1="25.4" x2="106.68" y2="27.94" width="0.1524" layer="91"/>
+<junction x="93.98" y="25.4"/>
+</segment>
+</net>
+<net name="N$6" class="0">
+<segment>
+<pinref part="U1" gate="G$1" pin="PB0"/>
+<wire x1="33.02" y1="63.5" x2="48.26" y2="63.5" width="0.1524" layer="91"/>
+<wire x1="48.26" y1="63.5" x2="48.26" y2="10.16" width="0.1524" layer="91"/>
+<pinref part="D17" gate="G$1" pin="C"/>
+<wire x1="48.26" y1="10.16" x2="63.5" y2="10.16" width="0.1524" layer="91"/>
+<wire x1="63.5" y1="10.16" x2="63.5" y2="12.7" width="0.1524" layer="91"/>
+<pinref part="D18" gate="G$1" pin="C"/>
+<wire x1="63.5" y1="10.16" x2="78.74" y2="10.16" width="0.1524" layer="91"/>
+<wire x1="78.74" y1="10.16" x2="78.74" y2="12.7" width="0.1524" layer="91"/>
+<junction x="63.5" y="10.16"/>
+</segment>
+</net>

Commit message: astro boy
Connections:
- net N$31: now also D10.A, D12.A, D13.A, D14.A, D15.A, D16.A, D18.A, D8.A, D9.A
Changed lines of the file:
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@@
 <wire x1="144.78" y1="86.36" x2="144.78" y2="53.34" width="0.1524" layer="91"/>
 <junction x="137.16" y="86.36"/>
+<wire x1="144.78" y1="53.34" x2="144.78" y2="35.56" width="0.1524" layer="91"/>
+<wire x1="144.78" y1="35.56" x2="144.78" y2="20.32" width="0.1524" layer="91"/>
+<pinref part="D16" gate="G$1" pin="A"/>
+<wire x1="137.16" y1="53.34" x2="144.78" y2="53.34" width="0.1524" layer="91"/>
+<junction x="144.78" y="53.34"/>
+<pinref part="D15" gate="G$1" pin="A"/>
+<wire x1="137.16" y1="53.34" x2="121.92" y2="53.34" width="0.1524" layer="91"/>
+<junction x="137.16" y="53.34"/>
+<pinref part="D14" gate="G$1" pin="A"/>
+<wire x1="121.92" y1="53.34" x2="106.68" y2="53.34" width="0.1524" layer="91"/>
+<junction x="121.92" y="53.34"/>
+<pinref part="D13" gate="G$1" pin="A"/>
+<wire x1="106.68" y1="53.34" x2="93.98" y2="53.34" width="0.1524" layer="91"/>
+<junction x="106.68" y="53.34"/>
+<pinref part="D12" gate="G$1" pin="A"/>
+<wire x1="93.98" y1="53.34" x2="78.74" y2="53.34" width="0.1524" layer="91"/>
+<junction x="93.98" y="53.34"/>
 <pinref part="D11" gate="G$1" pin="A"/>
-<wire x1="144.78" y1="53.34" x2="63.5" y2="53.34" width="0.1524" layer="91"/>
+<wire x1="78.74" y1="53.34" x2="63.5" y2="53.34" width="0.1524" layer="91"/>
+<junction x="78.74" y="53.34"/>
+<pinref part="D10" gate="G$1" pin="A"/>
+<wire x1="106.68" y1="35.56" x2="144.78" y2="35.56" width="0.1524" layer="91"/>
+<junction x="144.78" y="35.56"/>
+<pinref part="D9" gate="G$1" pin="A"/>
+<wire x1="106.68" y1="35.56" x2="93.98" y2="35.56" width="0.1524" layer="91"/>
+<junction x="106.68" y="35.56"/>
+<pinref part="D8" gate="G$1" pin="A"/>
+<wire x1="93.98" y1="35.56" x2="78.74" y2="35.56" width="0.1524" layer="91"/>
+<junction x="93.98" y="35.56"/>
 <pinref part="D7" gate="G$1" pin="A"/>
-<wire x1="144.78" y1="53.34" x2="144.78" y2="35.56" width="0.1524" layer="91"/>
-<wire x1="144.78" y1="35.56" x2="63.5" y2="35.56" width="0.1524" layer="91"/>
-<junction x="144.78" y="53.34"/>
-<wire x1="144.78" y1="35.56" x2="144.78" y2="20.32" width="0.1524" layer="91"/>
-<junction x="144.78" y="35.56"/>
+<wire x1="78.74" y1="35.56" x2="63.5" y2="35.56" width="0.1524" layer="91"/>
+<junction x="78.74" y="35.56"/>
+<pinref part="D18" gate="G$1" pin="A"/>
+<wire x1="78.74" y1="20.32" x2="144.78" y2="20.32" width="0.1524" layer="91"/>
 <pinref part="D17" gate="G$1" pin="A"/>
-<wire x1="144.78" y1="20.32" x2="63.5" y2="20.32" width="0.1524" layer="91"/>
+<wire x1="78.74" y1="20.32" x2="63.5" y2="20.32" width="0.1524" layer="91"/>
+<junction x="78.74" y="20.32"/>
 </segment>
 </net>
